File: KicadJE_SympleSeq.sch (KiCad schematic (older format))
At the start: 32 parts

Commit message: Counter w protection
Parts:
- removed C? (x2): 1u, Capacitor_SMD:C_1206_3216Metric_Pad1.42x1.75mm_HandSolder, symbol Device:C
- removed J?: In1.1, AJ-Dropbox-Kicad:PJ301SM, symbol Connector:AudioJack2_SwitchT
- removed J?: In1.2, AJ-Dropbox-Kicad:PJ301SM, symbol Connector:AudioJack2_SwitchT
- removed J?: Out1, AJ-Dropbox-Kicad:PJ301SM, symbol Connector:AudioJack2_SwitchT
- removed J?: In1.3, AJ-Dropbox-Kicad:PJ301SM, symbol Connector:AudioJack2_SwitchT
- removed P?: HEADER_2x5_Doepfer, Connector_IDC:IDC-Header_2x05_P2.54mm_Vertical, symbol Eurorack:HEADER_2x5_Doepfer
- removed R? (x3): 47k, Resistor_SMD:R_0805_2012Metric_Pad1.15x1.40mm_HandSolder, symbol Device:R
- removed R?: 4k7, Resistor_SMD:R_0805_2012Metric_Pad1.15x1.40mm_HandSolder, symbol Device:R
- removed U?: LM555, symbol Timer:LM555
- removed U?: 4017, symbol 4xxx:4017
- removed U?: TL082, symbol Amplifier_Operational:TL082
Connections:
- wire segments 100 -> 50
Other:
- moved on the sheet: R?, SW?, U?A, U?B
