File: KicadJE_SympleSeq.sch (KiCad schematic (older format))
At the start: 18 parts

Commit message: Sch taking form
Parts:
- added J?: Conn_01x06, symbol Connector_Generic:Conn_01x06
- added J? (x2): Conn_01x03, symbol Connector_Generic:Conn_01x03
Connections:
- net Control IO/CV: now also J?.1 (Pin_1), J?.1 (Pin_1)
- net Control IO/Gate: now also J?.2 (Pin_2), J?.2 (Pin_2)
- net Control IO/In_1: now also J?.5 (Pin_5)
- net Control IO/In_2: now also J?.4 (Pin_4)
- net Control IO/In_3: now also J?.3 (Pin_3)
- net Control IO/In_4: now also J?.2 (Pin_2)
- net Control IO/reset: now also J?.1 (Pin_1)
- net GND: now also J?.3 (Pin_3), J?.3 (Pin_3), J?.6 (Pin_6)
Changed lines of the file:
@@
 Wire Wire Line
 	1800 5500 1800 6100
+$Comp
+L Connector_Generic:Conn_01x06 J?
+U 1 1 5DAE9349
+P 6500 3600
+F 0 "J?" H 6418 4017 50  0000 C CNN
+F 1 "Conn_01x06" H 6418 3926 50  0000 C CNN
+F 2 "" H 6500 3600 50  0001 C CNN
+F 3 "~" H 6500 3600 50  0001 C CNN
+	1    6500 3600
+	-1   0    0    -1
+$EndComp
+$Comp
+L Connector_Generic:Conn_01x03 J?
+U 1 1 5DAEAEAF
+P 6500 4100
+F 0 "J?" H 6418 4417 50  0000 C CNN
+F 1 "Conn_01x03" H 6418 4326 50  0000 C CNN
+F 2 "" H 6500 4100 50  0001 C CNN
+F 3 "~" H 6500 4100 50  0001 C CNN
+	1    6500 4100
+	-1   0    0    -1
+$EndComp
+$Comp
+L Connector_Generic:Conn_01x03 J?
+U 1 1 5DAEBA5E
+P 6100 4100
+F 0 "J?" H 6018 4417 50  0000 C CNN
+F 1 "Conn_01x03" H 6018 4326 50  0000 C CNN
+F 2 "" H 6100 4100 50  0001 C CNN
+F 3 "~" H 6100 4100 50  0001 C CNN
+	1    6100 4100
+	-1   0    0    -1
+$EndComp
+Wire Wire Line
+	6700 4000 7000 4000
+Wire Wire Line
+	6700 4100 7000 4100
+Wire Wire Line
+	6700 3800 7000 3800
+Wire Wire Line
+	6700 3700 7000 3700
+Wire Wire Line
+	6700 3600 7000 3600
+Wire Wire Line
+	6700 3500 7000 3500
+Wire Wire Line
+	6700 3400 7000 3400
+Wire Wire Line
+	6300 4000 6700 4000
+Connection ~ 6700 4000
+Wire Wire Line
+	6300 4100 6700 4100
+Connection ~ 6700 4100
+Wire Wire Line
+	6300 4200 6700 4200
+$Comp
+L Envelope-cache-2018-08-04-13-00-04:GND #PWR?
+U 1 1 5DAF76B5
+P 6850 4300
+AR Path="/5DAF76B5" Ref="#PWR?"  Part="1"
+AR Path="/5C8C5FC0/5DAF76B5" Ref="#PWR?"  Part="1"
+F 0 "#PWR?" H 6850 4050 50  0001 C CNN
+F 1 "GND" H 6855 4127 50  0000 C CNN
+F 2 "" H 6850 4300 50  0001 C CNN
+F 3 "" H 6850 4300 50  0001 C CNN
+	1    6850 4300
+	1    0    0    -1
+$EndComp
+Wire Wire Line
+	6700 4200 6850 4200
+Wire Wire Line
+	6850 4200 6850 4300
+Connection ~ 6700 4200
+Wire Wire Line
+	6700 3900 6850 3900
+Wire Wire Line
+	6850 3900 6850 4200
+Connection ~ 6850 4200
 $EndSCHEMATC

Commit message: pin headers
Parts:
- removed J?: In2, AJ-Dropbox-Kicad:PJ301SM, symbol Connector:AudioJack2_SwitchT
- removed J?: Out2.1, AJ-Dropbox-Kicad:PJ301SM, symbol Connector:AudioJack2_SwitchT
- removed J?: Out2.3, AJ-Dropbox-Kicad:PJ301SM, symbol Connector:AudioJack2_SwitchT
- removed J?: Out2.2, AJ-Dropbox-Kicad:PJ301SM, symbol Connector:AudioJack2_SwitchT
- removed R?: 47k, Resistor_SMD:R_0805_2012Metric_Pad1.15x1.40mm_HandSolder, symbol Device:R
- removed R? (x3): 4k7, Resistor_SMD:R_0805_2012Metric_Pad1.15x1.40mm_HandSolder, symbol Device:R
- added J?: Reset + Step 1-4, symbol Connector_Generic:Conn_01x06
- added J?: Reset + Step 5-8, symbol Connector_Generic:Conn_01x06
- J?: value Conn_01x06 -> Reset + Step
- J?: value Conn_01x03 -> CV-G8_Mod2
- J?: value Conn_01x03 -> CV-G8_Mod1
Connections:
- net In1 is gone; now on net CV_M: SW?.2 (B)
- net In2 is gone; now on net G8_M: SW?.2 (B)
- net Clock/Q0: now also J?.2 (Pin_2)
- net Clock/Q1: now also J?.3 (Pin_3)
- net Clock/Q2: now also J?.4 (Pin_4)
- net Clock/Q3: now also J?.5 (Pin_5)
- net Clock/Q4: now also J?.2 (Pin_2)
- net Clock/Q5: now also J?.3 (Pin_3)
- net Clock/Q6: now also J?.4 (Pin_4)
- net Clock/Q7: now also J?.5 (Pin_5)
- net Clock/reset: now also J?.1 (Pin_1), J?.1 (Pin_1)
- net GND: now also J?.6 (Pin_6), J?.6 (Pin_6)
- net Control IO/CV renamed CV_M
- net Control IO/Gate renamed G8_M
Other:
- moved on the sheet: J?, R?, SW?, U?A, U?B

Commit message: base circuit done
Parts:
- removed R?: 20k, Resistor_SMD:R_0805_2012Metric_Pad1.15x1.40mm_HandSolder, symbol Device:R
- removed R? (x2): 47k, Resistor_SMD:R_0805_2012Metric_Pad1.15x1.40mm_HandSolder, symbol Device:R
- removed SW? (x2): Inv/NonInv, AJ-Dropbox-Kicad:SP1MS1, symbol Switch:SW_SPDT
- removed U?: TL082, AJ-Dropbox-Kicad:AJ_SO-8_5.3x6.2mm_P1.27mm, symbol Amplifier_Operational:TL082
- added J?: Clk_Hold, symbol Connector_Generic:Conn_01x03
- added J? (x2): CV-Out, symbol Connector_Generic:Conn_01x02
- added R? (x4): 1k, Resistor_SMD:R_0805_2012Metric_Pad1.15x1.40mm_HandSolder, symbol Device:R
- added R?: 47k, Resistor_SMD:R_0805_2012Metric_Pad1.15x1.40mm_HandSolder, symbol Device:R
- added R? (x2): 100k, Resistor_SMD:R_0805_2012Metric_Pad1.15x1.40mm_HandSolder, symbol Device:R
- added U?: TL082, symbol Amplifier_Operational:TL082
- R?: value 20k -> 47k
- R? (x2): value 47k -> 100k
Connections:
- net CV_M: now also R?.2, U?.5 (+)
- net Clock/clock_out: now also R?.1
- net Clock/hold: now also R?.1
- net G8_M: now also R?.2, U?.5 (+)
- net GND: now also J?.2 (Pin_2), J?.2 (Pin_2), J?.3 (Pin_3), R?.1, R?.2
- net Out2: no longer names the net of R?.1, U?.7
- net Out2: now also R?.2
- new net: J?.1 (Pin_1), R?.2
- new net: J?.2 (Pin_2), R?.2
- new net: J?.1 (Pin_1), R?.1 (x2)
- new net: R?.1, R?.2, U?.6 (-)
- new net: R?.1, R?.2, U?.7
Other:
- moved on the sheet: J?

Commit message: Annotate #1
Parts:
- J101, J106: renamed from J?; footprint (none) -> Connector_PinHeader_2.54mm:PinHeader_1x02_P2.54mm_Vertical
- J102, J107, J108: renamed from J?; footprint (none) -> Connector_PinHeader_2.54mm:PinHeader_1x06_P2.54mm_Vertical
- J103, J104, J105: renamed from J?; footprint (none) -> Connector_PinHeader_2.54mm:PinHeader_1x03_P2.54mm_Vertical
- gave numbers to parts that had none: 12

Commit message: control module PCB init
Parts:
- added unit 3 of U101
- U101: renamed from U102; footprint (none) -> AJ:AJ_SO-8_5.3x6.2mm_P1.27mm
- U101: footprint (none) -> AJ:AJ_SO-8_5.3x6.2mm_P1.27mm
Connections:
- net CV_M: now also U101.3 (+); no longer U101.5 (+)
- net at R101.1, R102.2: now also U101.2 (-); no longer U101.6 (-)
- net at R102.1, R103.2: now also U101.1; no longer U101.7
- new net +12Vc: U101.8 (V+)
- new net -12Vc: U101.4 (V-)
Changed lines of the file:
@@
 $EndSheet
 $Comp
-L Amplifier_Operational:TL082 U102
+L Amplifier_Operational:TL082 U101
 U 2 1 5D94A812
 P 2900 3500
-AR Path="/5D94A812" Ref="U102"  Part="2"
+AR Path="/5D94A812" Ref="U101"  Part="2"
 AR Path="/5C8C5FC0/5D94A812" Ref="U?"  Part="2"
-F 0 "U102" H 2900 3133 50  0000 C CNN
+F 0 "U101" H 2900 3133 50  0000 C CNN
 F 1 "TL082" H 2900 3224 50  0000 C CNN
-F 2 "" H 2900 3500 50  0001 C CNN
+F 2 "AJ:AJ_SO-8_5.3x6.2mm_P1.27mm" H 2900 3500 50  0001 C CNN
 F 3 "http://www.ti.com/lit/ds/symlink/tl081.pdf" H 2900 3500 50  0001 C CNN
 	2    2900 3500
@@
 $Comp
 L Amplifier_Operational:TL082 U101
-U 2 1 5DB86DE6
+U 1 1 5DB86DE6
 P 2900 1650
-AR Path="/5DB86DE6" Ref="U101"  Part="2"
+AR Path="/5DB86DE6" Ref="U101"  Part="1"
 AR Path="/5C8C5FC0/5DB86DE6" Ref="U?"  Part="2"
 F 0 "U101" H 2900 1283 50  0000 C CNN
 F 1 "TL082" H 2900 1374 50  0000 C CNN
-F 2 "" H 2900 1650 50  0001 C CNN
+F 2 "AJ:AJ_SO-8_5.3x6.2mm_P1.27mm" H 2900 1650 50  0001 C CNN
 F 3 "http://www.ti.com/lit/ds/symlink/tl081.pdf" H 2900 1650 50  0001 C CNN
-	2    2900 1650
+	1    2900 1650
 	1    0    0    1
 $EndComp
@@
 Wire Wire Line
 	3750 1650 3800 1650
+$Comp
+L Amplifier_Operational:TL082 U101
+U 3 1 5DBDC612
+P 6650 6900
+AR Path="/5DBDC612" Ref="U101"  Part="3"
+AR Path="/5C8C5FC0/5DBDC612" Ref="U?"  Part="3"
+F 0 "U101" H 6608 6946 50  0000 L CNN
+F 1 "TL082" H 6608 6855 50  0000 L CNN
+F 2 "AJ:AJ_SO-8_5.3x6.2mm_P1.27mm" H 6650 6900 50  0001 C CNN
+F 3 "http://www.ti.com/lit/ds/symlink/tl081.pdf" H 6650 6900 50  0001 C CNN
+	3    6650 6900
+	1    0    0    -1
+$EndComp
+Wire Wire Line
+	6550 6500 6550 6600
+Wire Wire Line
+	6550 7300 6550 7200
+Text GLabel 6550 6500 1    50   Input ~ 0
++12Vc
+Text GLabel 6550 7300 3    50   Input ~ 0
+-12Vc
 $EndSCHEMATC

Commit message: Init Clock board
Parts:
- J106: value CV-Out -> G8-Out
Changed lines of the file:
@@
 P 4000 3500
 F 0 "J106" H 4080 3492 50  0000 L CNN
-F 1 "CV-Out" H 4080 3401 50  0000 L CNN
+F 1 "G8-Out" H 4080 3401 50  0000 L CNN
 F 2 "Connector_PinHeader_2.54mm:PinHeader_1x02_P2.54mm_Vertical" H 4000 3500 50  0001 C CNN
 F 3 "~" H 4000 3500 50  0001 C CNN

Commit message: clock board done
Parts:
- added J109: CV-G8_Base, Connector_PinHeader_2.54mm:PinHeader_1x03_P2.54mm_Vertical, symbol Connector_Generic:Conn_01x03
Connections:
- net CV_M: now also J109.1 (Pin_1)
- net G8_M: now also J109.2 (Pin_2)
- net GND: now also J109.3 (Pin_3)
Changed lines of the file:
@@
 P 6150 2450
 F 0 "J104" H 6068 2767 50  0000 C CNN
-F 1 "CV-G8_Mod2" H 6068 2676 50  0000 C CNN
+F 1 "CV-G8_Mod2" H 6000 2700 50  0000 C CNN
 F 2 "Connector_PinHeader_2.54mm:PinHeader_1x03_P2.54mm_Vertical" H 6150 2450 50  0001 C CNN
 F 3 "~" H 6150 2450 50  0001 C CNN
@@
 Text GLabel 6550 7300 3    50   Input ~ 0
 -12Vc
+$Comp
+L Connector_Generic:Conn_01x03 J109
+U 1 1 5DC2EB18
+P 5350 2450
+F 0 "J109" H 5268 2767 50  0000 C CNN
+F 1 "CV-G8_Base" H 5400 2700 50  0000 C CNN
+F 2 "Connector_PinHeader_2.54mm:PinHeader_1x03_P2.54mm_Vertical" H 5350 2450 50  0001 C CNN
+F 3 "~" H 5350 2450 50  0001 C CNN
+	1    5350 2450
+	-1   0    0    -1
+$EndComp
+Wire Wire Line
+	5550 2450 5950 2450
+Wire Wire Line
+	5550 2550 5950 2550
+Wire Wire Line
+	5550 2350 5950 2350
+Connection ~ 5950 2350
+Connection ~ 5950 2450
+Connection ~ 5950 2550
 $EndSCHEMATC
