File: KicadJE_SympleSeq.sch (KiCad schematic (older format))
At the start: 30 parts, among them J101 CV-Out, J102 Reset + Step, J103 CV-G8_Mod1, J104 CV-G8_Mod2, J105 Clk_Hold, J106 G8-Out, J107 Reset + Step 1-4, J108 Reset + Step 5-8, J109 CV-G8_Base, U101 TL082

Commit message: slave clk - debounce hold etc
Parts:
- added C?: 100n, Capacitor_SMD:C_0805_2012Metric, symbol Device:C_Small
Connections:
- net G8_M: now also C?.2; no longer R110.2, U101.5 (+)
- new net: C?.1, R110.2, U101.5 (+)
Changed lines of the file:
@@
 	3500 3600 3500 3950
 Wire Wire Line
-	1850 3600 2500 3600
+	1850 3600 2100 3600
 $Comp
 L Amplifier_Operational:TL082 U101
@@
 Wire Wire Line
 	6850 4700 7000 4700
+$Comp
+L Device:C_Small C?
+U 1 1 5EAA1054
+P 2200 3600
+F 0 "C?" V 2175 3725 50  0000 C CNN
+F 1 "100n" V 2175 3475 50  0000 C CNN
+F 2 "Capacitor_SMD:C_0805_2012Metric" H 2200 3600 50  0001 C CNN
+F 3 "~" H 2200 3600 50  0001 C CNN
+	1    2200 3600
+	0    1    1    0
+$EndComp
+Wire Wire Line
+	2300 3600 2500 3600
 $EndSCHEMATC

Commit message: RevB updates
Parts:
- removed R? (x2): 1k, Resistor_SMD:R_0805_2012Metric_Pad1.15x1.40mm_HandSolder, symbol Device:R
- added D? (x2): LL4148, Diode_SMD:D_MiniMELF, symbol Diode:LL4148
- added D?: 5V1 Opt, Diode_SMD:D_MiniMELF, symbol Device:D_Zener_ALT
Connections:
- net Clock/hold: now also R108.1
- net Clock/reset: now also D?.1 (K), D?.1 (K)
- net GND: now also D?.2 (A)
- net at C?.1, R110.2, U101.5 (+): now also D?.1 (K)
- net at J107.1 (Pin_1): now also D?.2 (A)
- net at J108.1 (Pin_1): now also D?.2 (A)
Changed lines of the file:
@@
 $EndComp
 Wire Wire Line
-	2500 4100 2500 4000
+	2500 4100 2500 4075
 Wire Wire Line
 	2500 3700 2500 3600
@@
 	6625 3200 7000 3200
 Wire Wire Line
-	6625 3300 6975 3300
-Wire Wire Line
 	6575 3700 6650 3700
 Wire Wire Line
@@
 Wire Wire Line
 	6900 4300 6900 3600
-Connection ~ 6900 3600
 Wire Wire Line
 	6900 3600 7000 3600
@@
 Wire Wire Line
 	6575 3600 6600 3600
-$Comp
-L Device:R R?
-U 1 1 5EA9CB60
-P 6750 3600
-AR Path="/5EA9CB60" Ref="R?"  Part="1"
-AR Path="/5C8C5FC0/5EA9CB60" Ref="R?"  Part="1"
-F 0 "R?" V 6700 3750 50  0000 C CNN
-F 1 "1k" V 6750 3600 50  0000 C CNN
-F 2 "Resistor_SMD:R_0805_2012Metric_Pad1.15x1.40mm_HandSolder" V 6680 3600 50  0001 C CNN
-F 3 "~" H 6750 3600 50  0001 C CNN
-	1    6750 3600
-	0    1    1    0
-$EndComp
-$Comp
-L Device:R R?
-U 1 1 5EA9CD71
-P 6750 4300
-AR Path="/5EA9CD71" Ref="R?"  Part="1"
-AR Path="/5C8C5FC0/5EA9CD71" Ref="R?"  Part="1"
-F 0 "R?" V 6700 4450 50  0000 C CNN
-F 1 "1k" V 6750 4300 50  0000 C CNN
-F 2 "Resistor_SMD:R_0805_2012Metric_Pad1.15x1.40mm_HandSolder" V 6680 4300 50  0001 C CNN
-F 3 "~" H 6750 4300 50  0001 C CNN
-	1    6750 4300
-	0    1    1    0
-$EndComp
 $Comp
 L Device:C_Small C?
@@
 $EndComp
 Wire Wire Line
-	2300 3600 2500 3600
+	2300 3600 2350 3600
+Wire Wire Line
+	6625 3300 7000 3300
+$Comp
+L Diode:LL4148 D?
+U 1 1 5EBDB059
+P 6750 4300
+AR Path="/5C8BFBBC/5EBDB059" Ref="D?"  Part="1"
+AR Path="/5EBDB059" Ref="D?"  Part="1"
+F 0 "D?" H 6925 4275 50  0000 C CNN
+F 1 "LL4148" H 6550 4250 50  0000 C CNN
+F 2 "Diode_SMD:D_MiniMELF" H 6750 4125 50  0001 C CNN
+F 3 "http://www.vishay.com/docs/85557/ll4148.pdf" H 6750 4300 50  0001 C CNN
+	1    6750 4300
+	-1   0    0    1
+$EndComp
+$Comp
+L Diode:LL4148 D?
+U 1 1 5EBDDE8B
+P 6750 3600
+AR Path="/5C8BFBBC/5EBDDE8B" Ref="D?"  Part="1"
+AR Path="/5EBDDE8B" Ref="D?"  Part="1"
+F 0 "D?" H 6925 3575 50  0000 C CNN
+F 1 "LL4148" H 6550 3550 50  0000 C CNN
+F 2 "Diode_SMD:D_MiniMELF" H 6750 3425 50  0001 C CNN
+F 3 "http://www.vishay.com/docs/85557/ll4148.pdf" H 6750 3600 50  0001 C CNN
+	1    6750 3600
+	-1   0    0    1
+$EndComp
+Connection ~ 6900 3600
+$Comp
+L Device:D_Zener_ALT D?
+U 1 1 5EBE23F1
+P 2350 3850
+AR Path="/5C8BFBBC/5EBE23F1" Ref="D?"  Part="1"
+AR Path="/5EBE23F1" Ref="D?"  Part="1"
+F 0 "D?" H 2600 3775 50  0000 C CNN
+F 1 "5V1 Opt" H 2350 3750 50  0000 C CNN
+F 2 "Diode_SMD:D_MiniMELF" H 2350 3675 50  0001 C CNN
+F 3 "http://www.vishay.com/docs/85557/ll4148.pdf" H 2350 3850 50  0001 C CNN
+	1    2350 3850
+	0    1    1    0
+$EndComp
+Wire Wire Line
+	2350 4000 2350 4075
+Wire Wire Line
+	2350 4075 2500 4075
+Connection ~ 2500 4075
+Wire Wire Line
+	2500 4075 2500 4000
+Wire Wire Line
+	2350 3700 2350 3600
+Connection ~ 2350 3600
+Wire Wire Line
+	2350 3600 2500 3600
 $EndSCHEMATC

Commit message: ERC Rev B
Parts:
- gave numbers to parts that had none: 12
Changed lines of the file:
@@
 	6575 3600 6600 3600
 $Comp
-L Device:C_Small C?
+L Device:C_Small C102
 U 1 1 5EA9D3AA
 P 6750 3700
-F 0 "C?" V 6725 3825 50  0000 C CNN
+F 0 "C102" V 6725 3825 50  0000 C CNN
 F 1 "100n" V 6725 3575 50  0000 C CNN
 F 2 "Capacitor_SMD:C_0805_2012Metric" H 6750 3700 50  0001 C CNN
@@
 	6575 3800 6650 3800
 $Comp
-L Device:C_Small C?
+L Device:C_Small C103
 U 1 1 5EA9ECF0
 P 6750 3800
-F 0 "C?" V 6725 3925 50  0000 C CNN
+F 0 "C103" V 6725 3925 50  0000 C CNN
 F 1 "100n" V 6725 3675 50  0000 C CNN
 F 2 "Capacitor_SMD:C_0805_2012Metric" H 6750 3800 50  0001 C CNN
@@
 	6850 3800 7000 3800
 $Comp
-L Device:C_Small C?
+L Device:C_Small C104
 U 1 1 5EA9F088
 P 6750 3900
-F 0 "C?" V 6725 4025 50  0000 C CNN
+F 0 "C104" V 6725 4025 50  0000 C CNN
 F 1 "100n" V 6725 3775 50  0000 C CNN
 F 2 "Capacitor_SMD:C_0805_2012Metric" H 6750 3900 50  0001 C CNN
@@
 	6850 3900 7000 3900
 $Comp
-L Device:C_Small C?
+L Device:C_Small C105
 U 1 1 5EA9F2B1
 P 6750 4000
-F 0 "C?" V 6725 4125 50  0000 C CNN
+F 0 "C105" V 6725 4125 50  0000 C CNN
 F 1 "100n" V 6725 3875 50  0000 C CNN
 F 2 "Capacitor_SMD:C_0805_2012Metric" H 6750 4000 50  0001 C CNN
@@
 	6850 4000 7000 4000
 $Comp
-L Device:C_Small C?
+L Device:C_Small C106
 U 1 1 5EA9F4B3
 P 6750 4400
-F 0 "C?" V 6725 4525 50  0000 C CNN
+F 0 "C106" V 6725 4525 50  0000 C CNN
 F 1 "100n" V 6725 4275 50  0000 C CNN
 F 2 "Capacitor_SMD:C_0805_2012Metric" H 6750 4400 50  0001 C CNN
@@
 	6850 4400 7000 4400
 $Comp
-L Device:C_Small C?
+L Device:C_Small C107
 U 1 1 5EA9F9A4
 P 6750 4500
-F 0 "C?" V 6725 4625 50  0000 C CNN
+F 0 "C107" V 6725 4625 50  0000 C CNN
 F 1 "100n" V 6725 4375 50  0000 C CNN
 F 2 "Capacitor_SMD:C_0805_2012Metric" H 6750 4500 50  0001 C CNN
@@
 	6850 4500 7000 4500
 $Comp
-L Device:C_Small C?
+L Device:C_Small C108
 U 1 1 5EA9FCDB
 P 6750 4600
-F 0 "C?" V 6725 4725 50  0000 C CNN
+F 0 "C108" V 6725 4725 50  0000 C CNN
 F 1 "100n" V 6725 4475 50  0000 C CNN
 F 2 "Capacitor_SMD:C_0805_2012Metric" H 6750 4600 50  0001 C CNN
@@
 	6850 4600 7000 4600
 $Comp
-L Device:C_Small C?
+L Device:C_Small C109
 U 1 1 5EA9FEC4
 P 6750 4700
-F 0 "C?" V 6725 4825 50  0000 C CNN
+F 0 "C109" V 6725 4825 50  0000 C CNN
 F 1 "100n" V 6725 4575 50  0000 C CNN
 F 2 "Capacitor_SMD:C_0805_2012Metric" H 6750 4700 50  0001 C CNN
@@
 	6850 4700 7000 4700
 $Comp
-L Device:C_Small C?
+L Device:C_Small C101
 U 1 1 5EAA1054
 P 2200 3600
-F 0 "C?" V 2175 3725 50  0000 C CNN
+F 0 "C101" V 2175 3725 50  0000 C CNN
 F 1 "100n" V 2175 3475 50  0000 C CNN
 F 2 "Capacitor_SMD:C_0805_2012Metric" H 2200 3600 50  0001 C CNN
@@
 P 6750 4300
 AR Path="/5C8BFBBC/5EBDB059" Ref="D?"  Part="1"
-AR Path="/5EBDB059" Ref="D?"  Part="1"
-F 0 "D?" H 6925 4275 50  0000 C CNN
+AR Path="/5EBDB059" Ref="D103"  Part="1"
+F 0 "D103" H 6925 4275 50  0000 C CNN
 F 1 "LL4148" H 6550 4250 50  0000 C CNN
 F 2 "Diode_SMD:D_MiniMELF" H 6750 4125 50  0001 C CNN
@@
 P 6750 3600
 AR Path="/5C8BFBBC/5EBDDE8B" Ref="D?"  Part="1"
-AR Path="/5EBDDE8B" Ref="D?"  Part="1"
-F 0 "D?" H 6925 3575 50  0000 C CNN
+AR Path="/5EBDDE8B" Ref="D102"  Part="1"
+F 0 "D102" H 6925 3575 50  0000 C CNN
 F 1 "LL4148" H 6550 3550 50  0000 C CNN
 F 2 "Diode_SMD:D_MiniMELF" H 6750 3425 50  0001 C CNN
@@
 P 2350 3850
 AR Path="/5C8BFBBC/5EBE23F1" Ref="D?"  Part="1"
-AR Path="/5EBE23F1" Ref="D?"  Part="1"
-F 0 "D?" H 2600 3775 50  0000 C CNN
+AR Path="/5EBE23F1" Ref="D101"  Part="1"
+F 0 "D101" H 2600 3775 50  0000 C CNN
 F 1 "5V1 Opt" H 2350 3750 50  0000 C CNN
 F 2 "Diode_SMD:D_MiniMELF" H 2350 3675 50  0001 C CNN

Commit message: AJ Footprints
Parts:
- C101, C102, C103, C104, C105, C106, C107, C108, C109: footprint Capacitor_SMD:C_0805_2012Metric -> AJ:C_0805_2012Metric_Pad1.15x1.40mm_HandSolder
- R101, R102, R103, R104, R105, R106, R107, R108, R109, R110: footprint Resistor_SMD:R_0805_2012Metric_Pad1.15x1.40mm_HandSolder -> AJ:R_0805_2012Metric_Pad1.15x1.40mm_HandSolder
Changed lines of the file:
@@
 F 0 "R106" V 2693 3000 50  0000 C CNN
 F 1 "47k" V 2784 3000 50  0000 C CNN
-F 2 "Resistor_SMD:R_0805_2012Metric_Pad1.15x1.40mm_HandSolder" V 2830 3000 50  0001 C CNN
+F 2 "AJ:R_0805_2012Metric_Pad1.15x1.40mm_HandSolder" V 2830 3000 50  0001 C CNN
 F 3 "~" H 2900 3000 50  0001 C CNN
 	1    2900 3000
@@
 F 0 "R105" V 1693 3000 50  0000 C CNN
 F 1 "100k" V 1784 3000 50  0000 C CNN
-F 2 "Resistor_SMD:R_0805_2012Metric_Pad1.15x1.40mm_HandSolder" V 1830 3000 50  0001 C CNN
+F 2 "AJ:R_0805_2012Metric_Pad1.15x1.40mm_HandSolder" V 1830 3000 50  0001 C CNN
 F 3 "~" H 1900 3000 50  0001 C CNN
 	1    1900 3000
@@
 F 0 "R110" V 2293 3850 50  0000 C CNN
 F 1 "100k" V 2384 3850 50  0000 C CNN
-F 2 "Resistor_SMD:R_0805_2012Metric_Pad1.15x1.40mm_HandSolder" V 2430 3850 50  0001 C CNN
+F 2 "AJ:R_0805_2012Metric_Pad1.15x1.40mm_HandSolder" V 2430 3850 50  0001 C CNN
 F 3 "~" H 2500 3850 50  0001 C CNN
 	1    2500 3850
@@
 F 0 "R107" V 6425 3350 50  0000 C CNN
 F 1 "1k" V 6475 3200 50  0000 C CNN
-F 2 "Resistor_SMD:R_0805_2012Metric_Pad1.15x1.40mm_HandSolder" V 6405 3200 50  0001 C CNN
+F 2 "AJ:R_0805_2012Metric_Pad1.15x1.40mm_HandSolder" V 6405 3200 50  0001 C CNN
 F 3 "~" H 6475 3200 50  0001 C CNN
 	1    6475 3200
@@
 F 0 "R108" V 6425 3450 50  0000 C CNN
 F 1 "1k" V 6475 3300 50  0000 C CNN
-F 2 "Resistor_SMD:R_0805_2012Metric_Pad1.15x1.40mm_HandSolder" V 6405 3300 50  0001 C CNN
+F 2 "AJ:R_0805_2012Metric_Pad1.15x1.40mm_HandSolder" V 6405 3300 50  0001 C CNN
 F 3 "~" H 6475 3300 50  0001 C CNN
 	1    6475 3300
@@
 F 0 "R102" V 2693 1150 50  0000 C CNN
 F 1 "47k" V 2784 1150 50  0000 C CNN
-F 2 "Resistor_SMD:R_0805_2012Metric_Pad1.15x1.40mm_HandSolder" V 2830 1150 50  0001 C CNN
+F 2 "AJ:R_0805_2012Metric_Pad1.15x1.40mm_HandSolder" V 2830 1150 50  0001 C CNN
 F 3 "~" H 2900 1150 50  0001 C CNN
 	1    2900 1150
@@
 F 0 "R104" V 2293 2000 50  0000 C CNN
 F 1 "100k" V 2384 2000 50  0000 C CNN
-F 2 "Resistor_SMD:R_0805_2012Metric_Pad1.15x1.40mm_HandSolder" V 2430 2000 50  0001 C CNN
+F 2 "AJ:R_0805_2012Metric_Pad1.15x1.40mm_HandSolder" V 2430 2000 50  0001 C CNN
 F 3 "~" H 2500 2000 50  0001 C CNN
 	1    2500 2000
@@
 F 0 "R101" V 1693 1150 50  0000 C CNN
 F 1 "100k" V 1784 1150 50  0000 C CNN
-F 2 "Resistor_SMD:R_0805_2012Metric_Pad1.15x1.40mm_HandSolder" V 1830 1150 50  0001 C CNN
+F 2 "AJ:R_0805_2012Metric_Pad1.15x1.40mm_HandSolder" V 1830 1150 50  0001 C CNN
 F 3 "~" H 1900 1150 50  0001 C CNN
 	1    1900 1150
@@
 F 0 "R109" V 3550 3650 50  0000 C CNN
 F 1 "1k" V 3600 3500 50  0000 C CNN
-F 2 "Resistor_SMD:R_0805_2012Metric_Pad1.15x1.40mm_HandSolder" V 3530 3500 50  0001 C CNN
+F 2 "AJ:R_0805_2012Metric_Pad1.15x1.40mm_HandSolder" V 3530 3500 50  0001 C CNN
 F 3 "~" H 3600 3500 50  0001 C CNN
 	1    3600 3500
@@
 F 0 "R103" V 3550 1800 50  0000 C CNN
 F 1 "1k" V 3600 1650 50  0000 C CNN
-F 2 "Resistor_SMD:R_0805_2012Metric_Pad1.15x1.40mm_HandSolder" V 3530 1650 50  0001 C CNN
+F 2 "AJ:R_0805_2012Metric_Pad1.15x1.40mm_HandSolder" V 3530 1650 50  0001 C CNN
 F 3 "~" H 3600 1650 50  0001 C CNN
 	1    3600 1650
@@
 F 0 "C102" V 6725 3825 50  0000 C CNN
 F 1 "100n" V 6725 3575 50  0000 C CNN
-F 2 "Capacitor_SMD:C_0805_2012Metric" H 6750 3700 50  0001 C CNN
+F 2 "AJ:C_0805_2012Metric_Pad1.15x1.40mm_HandSolder" H 6750 3700 50  0001 C CNN
 F 3 "~" H 6750 3700 50  0001 C CNN
 	1    6750 3700
@@
 F 0 "C103" V 6725 3925 50  0000 C CNN
 F 1 "100n" V 6725 3675 50  0000 C CNN
-F 2 "Capacitor_SMD:C_0805_2012Metric" H 6750 3800 50  0001 C CNN
+F 2 "AJ:C_0805_2012Metric_Pad1.15x1.40mm_HandSolder" H 6750 3800 50  0001 C CNN
 F 3 "~" H 6750 3800 50  0001 C CNN
 	1    6750 3800
@@
 F 0 "C104" V 6725 4025 50  0000 C CNN
 F 1 "100n" V 6725 3775 50  0000 C CNN
-F 2 "Capacitor_SMD:C_0805_2012Metric" H 6750 3900 50  0001 C CNN
+F 2 "AJ:C_0805_2012Metric_Pad1.15x1.40mm_HandSolder" H 6750 3900 50  0001 C CNN
 F 3 "~" H 6750 3900 50  0001 C CNN
 	1    6750 3900
@@
 F 0 "C105" V 6725 4125 50  0000 C CNN
 F 1 "100n" V 6725 3875 50  0000 C CNN
-F 2 "Capacitor_SMD:C_0805_2012Metric" H 6750 4000 50  0001 C CNN
+F 2 "AJ:C_0805_2012Metric_Pad1.15x1.40mm_HandSolder" H 6750 4000 50  0001 C CNN
 F 3 "~" H 6750 4000 50  0001 C CNN
 	1    6750 4000
@@
 F 0 "C106" V 6725 4525 50  0000 C CNN
 F 1 "100n" V 6725 4275 50  0000 C CNN
-F 2 "Capacitor_SMD:C_0805_2012Metric" H 6750 4400 50  0001 C CNN
+F 2 "AJ:C_0805_2012Metric_Pad1.15x1.40mm_HandSolder" H 6750 4400 50  0001 C CNN
 F 3 "~" H 6750 4400 50  0001 C CNN
 	1    6750 4400
@@
 F 0 "C107" V 6725 4625 50  0000 C CNN
 F 1 "100n" V 6725 4375 50  0000 C CNN
-F 2 "Capacitor_SMD:C_0805_2012Metric" H 6750 4500 50  0001 C CNN
+F 2 "AJ:C_0805_2012Metric_Pad1.15x1.40mm_HandSolder" H 6750 4500 50  0001 C CNN
 F 3 "~" H 6750 4500 50  0001 C CNN
 	1    6750 4500
@@
 F 0 "C108" V 6725 4725 50  0000 C CNN
 F 1 "100n" V 6725 4475 50  0000 C CNN
-F 2 "Capacitor_SMD:C_0805_2012Metric" H 6750 4600 50  0001 C CNN
+F 2 "AJ:C_0805_2012Metric_Pad1.15x1.40mm_HandSolder" H 6750 4600 50  0001 C CNN
 F 3 "~" H 6750 4600 50  0001 C CNN
 	1    6750 4600
@@
 F 0 "C109" V 6725 4825 50  0000 C CNN
 F 1 "100n" V 6725 4575 50  0000 C CNN
-F 2 "Capacitor_SMD:C_0805_2012Metric" H 6750 4700 50  0001 C CNN
+F 2 "AJ:C_0805_2012Metric_Pad1.15x1.40mm_HandSolder" H 6750 4700 50  0001 C CNN
 F 3 "~" H 6750 4700 50  0001 C CNN
 	1    6750 4700
@@
 F 0 "C101" V 2175 3725 50  0000 C CNN
 F 1 "100n" V 2175 3475 50  0000 C CNN
-F 2 "Capacitor_SMD:C_0805_2012Metric" H 2200 3600 50  0001 C CNN
+F 2 "AJ:C_0805_2012Metric_Pad1.15x1.40mm_HandSolder" H 2200 3600 50  0001 C CNN
 F 3 "~" H 2200 3600 50  0001 C CNN
 	1    2200 3600

Commit message: AJ footprints updated
Parts:
- C101, C102, C103, C104, C105, C106, C107, C108, C109: footprint AJ:C_0805_2012Metric_Pad1.15x1.40mm_HandSolder -> AJ:C_0805_AJ
- R101, R102, R103, R104, R105, R106, R107, R108, R109, R110: footprint AJ:R_0805_2012Metric_Pad1.15x1.40mm_HandSolder -> AJ:R_0805_AJ
Changed lines of the file:
@@
 F 0 "R106" V 2693 3000 50  0000 C CNN
 F 1 "47k" V 2784 3000 50  0000 C CNN
-F 2 "AJ:R_0805_2012Metric_Pad1.15x1.40mm_HandSolder" V 2830 3000 50  0001 C CNN
+F 2 "AJ:R_0805_AJ" V 2830 3000 50  0001 C CNN
 F 3 "~" H 2900 3000 50  0001 C CNN
 	1    2900 3000
@@
 F 0 "R105" V 1693 3000 50  0000 C CNN
 F 1 "100k" V 1784 3000 50  0000 C CNN
-F 2 "AJ:R_0805_2012Metric_Pad1.15x1.40mm_HandSolder" V 1830 3000 50  0001 C CNN
+F 2 "AJ:R_0805_AJ" V 1830 3000 50  0001 C CNN
 F 3 "~" H 1900 3000 50  0001 C CNN
 	1    1900 3000
@@
 F 0 "R110" V 2293 3850 50  0000 C CNN
 F 1 "100k" V 2384 3850 50  0000 C CNN
-F 2 "AJ:R_0805_2012Metric_Pad1.15x1.40mm_HandSolder" V 2430 3850 50  0001 C CNN
+F 2 "AJ:R_0805_AJ" V 2430 3850 50  0001 C CNN
 F 3 "~" H 2500 3850 50  0001 C CNN
 	1    2500 3850
@@
 F 0 "R107" V 6425 3350 50  0000 C CNN
 F 1 "1k" V 6475 3200 50  0000 C CNN
-F 2 "AJ:R_0805_2012Metric_Pad1.15x1.40mm_HandSolder" V 6405 3200 50  0001 C CNN
+F 2 "AJ:R_0805_AJ" V 6405 3200 50  0001 C CNN
 F 3 "~" H 6475 3200 50  0001 C CNN
 	1    6475 3200
@@
 F 0 "R108" V 6425 3450 50  0000 C CNN
 F 1 "1k" V 6475 3300 50  0000 C CNN
-F 2 "AJ:R_0805_2012Metric_Pad1.15x1.40mm_HandSolder" V 6405 3300 50  0001 C CNN
+F 2 "AJ:R_0805_AJ" V 6405 3300 50  0001 C CNN
 F 3 "~" H 6475 3300 50  0001 C CNN
 	1    6475 3300
@@
 F 0 "R102" V 2693 1150 50  0000 C CNN
 F 1 "47k" V 2784 1150 50  0000 C CNN
-F 2 "AJ:R_0805_2012Metric_Pad1.15x1.40mm_HandSolder" V 2830 1150 50  0001 C CNN
+F 2 "AJ:R_0805_AJ" V 2830 1150 50  0001 C CNN
 F 3 "~" H 2900 1150 50  0001 C CNN
 	1    2900 1150
@@
 F 0 "R104" V 2293 2000 50  0000 C CNN
 F 1 "100k" V 2384 2000 50  0000 C CNN
-F 2 "AJ:R_0805_2012Metric_Pad1.15x1.40mm_HandSolder" V 2430 2000 50  0001 C CNN
+F 2 "AJ:R_0805_AJ" V 2430 2000 50  0001 C CNN
 F 3 "~" H 2500 2000 50  0001 C CNN
 	1    2500 2000
@@
 F 0 "R101" V 1693 1150 50  0000 C CNN
 F 1 "100k" V 1784 1150 50  0000 C CNN
-F 2 "AJ:R_0805_2012Metric_Pad1.15x1.40mm_HandSolder" V 1830 1150 50  0001 C CNN
+F 2 "AJ:R_0805_AJ" V 1830 1150 50  0001 C CNN
 F 3 "~" H 1900 1150 50  0001 C CNN
 	1    1900 1150
@@
 F 0 "R109" V 3550 3650 50  0000 C CNN
 F 1 "1k" V 3600 3500 50  0000 C CNN
-F 2 "AJ:R_0805_2012Metric_Pad1.15x1.40mm_HandSolder" V 3530 3500 50  0001 C CNN
+F 2 "AJ:R_0805_AJ" V 3530 3500 50  0001 C CNN
 F 3 "~" H 3600 3500 50  0001 C CNN
 	1    3600 3500
@@
 F 0 "R103" V 3550 1800 50  0000 C CNN
 F 1 "1k" V 3600 1650 50  0000 C CNN
-F 2 "AJ:R_0805_2012Metric_Pad1.15x1.40mm_HandSolder" V 3530 1650 50  0001 C CNN
+F 2 "AJ:R_0805_AJ" V 3530 1650 50  0001 C CNN
 F 3 "~" H 3600 1650 50  0001 C CNN
 	1    3600 1650
@@
 F 0 "C102" V 6725 3825 50  0000 C CNN
 F 1 "100n" V 6725 3575 50  0000 C CNN
-F 2 "AJ:C_0805_2012Metric_Pad1.15x1.40mm_HandSolder" H 6750 3700 50  0001 C CNN
+F 2 "AJ:C_0805_AJ" H 6750 3700 50  0001 C CNN
 F 3 "~" H 6750 3700 50  0001 C CNN
 	1    6750 3700
@@
 F 0 "C103" V 6725 3925 50  0000 C CNN
 F 1 "100n" V 6725 3675 50  0000 C CNN
-F 2 "AJ:C_0805_2012Metric_Pad1.15x1.40mm_HandSolder" H 6750 3800 50  0001 C CNN
+F 2 "AJ:C_0805_AJ" H 6750 3800 50  0001 C CNN
 F 3 "~" H 6750 3800 50  0001 C CNN
 	1    6750 3800
@@
 F 0 "C104" V 6725 4025 50  0000 C CNN
 F 1 "100n" V 6725 3775 50  0000 C CNN
-F 2 "AJ:C_0805_2012Metric_Pad1.15x1.40mm_HandSolder" H 6750 3900 50  0001 C CNN
+F 2 "AJ:C_0805_AJ" H 6750 3900 50  0001 C CNN
 F 3 "~" H 6750 3900 50  0001 C CNN
 	1    6750 3900
@@
 F 0 "C105" V 6725 4125 50  0000 C CNN
 F 1 "100n" V 6725 3875 50  0000 C CNN
-F 2 "AJ:C_0805_2012Metric_Pad1.15x1.40mm_HandSolder" H 6750 4000 50  0001 C CNN
+F 2 "AJ:C_0805_AJ" H 6750 4000 50  0001 C CNN
 F 3 "~" H 6750 4000 50  0001 C CNN
 	1    6750 4000
@@
 F 0 "C106" V 6725 4525 50  0000 C CNN
 F 1 "100n" V 6725 4275 50  0000 C CNN
-F 2 "AJ:C_0805_2012Metric_Pad1.15x1.40mm_HandSolder" H 6750 4400 50  0001 C CNN
+F 2 "AJ:C_0805_AJ" H 6750 4400 50  0001 C CNN
 F 3 "~" H 6750 4400 50  0001 C CNN
 	1    6750 4400
@@
 F 0 "C107" V 6725 4625 50  0000 C CNN
 F 1 "100n" V 6725 4375 50  0000 C CNN
-F 2 "AJ:C_0805_2012Metric_Pad1.15x1.40mm_HandSolder" H 6750 4500 50  0001 C CNN
+F 2 "AJ:C_0805_AJ" H 6750 4500 50  0001 C CNN
 F 3 "~" H 6750 4500 50  0001 C CNN
 	1    6750 4500
@@
 F 0 "C108" V 6725 4725 50  0000 C CNN
 F 1 "100n" V 6725 4475 50  0000 C CNN
-F 2 "AJ:C_0805_2012Metric_Pad1.15x1.40mm_HandSolder" H 6750 4600 50  0001 C CNN
+F 2 "AJ:C_0805_AJ" H 6750 4600 50  0001 C CNN
 F 3 "~" H 6750 4600 50  0001 C CNN
 	1    6750 4600
@@
 F 0 "C109" V 6725 4825 50  0000 C CNN
 F 1 "100n" V 6725 4575 50  0000 C CNN
-F 2 "AJ:C_0805_2012Metric_Pad1.15x1.40mm_HandSolder" H 6750 4700 50  0001 C CNN
+F 2 "AJ:C_0805_AJ" H 6750 4700 50  0001 C CNN
 F 3 "~" H 6750 4700 50  0001 C CNN
 	1    6750 4700
@@
 F 0 "C101" V 2175 3725 50  0000 C CNN
 F 1 "100n" V 2175 3475 50  0000 C CNN
-F 2 "AJ:C_0805_2012Metric_Pad1.15x1.40mm_HandSolder" H 2200 3600 50  0001 C CNN
+F 2 "AJ:C_0805_AJ" H 2200 3600 50  0001 C CNN
 F 3 "~" H 2200 3600 50  0001 C CNN
 	1    2200 3600

Commit message: hold/rst
Parts:
- J105: value Clk_Hold -> Hold_Rst
Connections:
- net Clock/clock_out: no longer R107.1
- net Clock/hold: now also R107.1; no longer R108.1
- net Clock/reset: now also R108.1
Other:
- moved on the sheet: J105, R107, R108
Changed lines of the file:
@@
 U 1 1 5DAFAB5F
 P 6375 3800
-F 0 "J107" H 6293 4217 50  0000 C CNN
+F 0 "J107" H 6525 4025 50  0000 C CNN
 F 1 "Reset + Step 1-4" H 6293 4126 50  0000 C CNN
 F 2 "Connector_PinHeader_2.54mm:PinHeader_1x06_P2.54mm_Vertical" H 6375 3800 50  0001 C CNN
@@
 L Connector_Generic:Conn_01x03 J105
 U 1 1 5DB6936A
-P 5875 3300
-F 0 "J105" H 5793 3617 50  0000 C CNN
-F 1 "Clk_Hold" H 5793 3526 50  0000 C CNN
-F 2 "Connector_PinHeader_2.54mm:PinHeader_1x03_P2.54mm_Vertical" H 5875 3300 50  0001 C CNN
-F 3 "~" H 5875 3300 50  0001 C CNN
-	1    5875 3300
+P 5750 3400
+F 0 "J105" H 5668 3717 50  0000 C CNN
+F 1 "Hold_Rst" H 5668 3626 50  0000 C CNN
+F 2 "Connector_PinHeader_2.54mm:PinHeader_1x03_P2.54mm_Vertical" H 5750 3400 50  0001 C CNN
+F 3 "~" H 5750 3400 50  0001 C CNN
+	1    5750 3400
 	-1   0    0    -1
 $EndComp
 Wire Wire Line
-	6075 3300 6325 3300
-Wire Wire Line
-	6075 3200 6325 3200
+	5950 3400 6200 3400
+Wire Wire Line
+	5950 3300 6200 3300
 $Comp
 L Envelope-cache-2018-08-04-13-00-04:GND #PWR0107
 U 1 1 5DB715F6
-P 6125 3500
+P 6000 3600
 AR Path="/5DB715F6" Ref="#PWR0107"  Part="1"
 AR Path="/5C8C5FC0/5DB715F6" Ref="#PWR?"  Part="1"
-F 0 "#PWR0107" H 6125 3250 50  0001 C CNN
-F 1 "GND" H 6130 3327 50  0000 C CNN
-F 2 "" H 6125 3500 50  0001 C CNN
-F 3 "" H 6125 3500 50  0001 C CNN
-	1    6125 3500
-	1    0    0    -1
-$EndComp
-Wire Wire Line
-	6075 3400 6125 3400
-Wire Wire Line
-	6125 3400 6125 3500
+F 0 "#PWR0107" H 6000 3350 50  0001 C CNN
+F 1 "GND" H 6005 3427 50  0000 C CNN
+F 2 "" H 6000 3600 50  0001 C CNN
+F 3 "" H 6000 3600 50  0001 C CNN
+	1    6000 3600
+	1    0    0    -1
+$EndComp
+Wire Wire Line
+	5950 3500 6000 3500
+Wire Wire Line
+	6000 3500 6000 3600
 $Comp
 L Device:R R107
 U 1 1 5DB7317B
-P 6475 3200
+P 6350 3300
 AR Path="/5DB7317B" Ref="R107"  Part="1"
 AR Path="/5C8C5FC0/5DB7317B" Ref="R?"  Part="1"
-F 0 "R107" V 6425 3350 50  0000 C CNN
-F 1 "1k" V 6475 3200 50  0000 C CNN
-F 2 "AJ:R_0805_AJ" V 6405 3200 50  0001 C CNN
-F 3 "~" H 6475 3200 50  0001 C CNN
-	1    6475 3200
+F 0 "R107" V 6300 3100 50  0000 C CNN
+F 1 "1k" V 6350 3300 50  0000 C CNN
+F 2 "AJ:R_0805_AJ" V 6280 3300 50  0001 C CNN
+F 3 "~" H 6350 3300 50  0001 C CNN
+	1    6350 3300
 	0    1    1    0
 $EndComp
@@
 L Device:R R108
 U 1 1 5DB73B0A
-P 6475 3300
+P 6350 3400
 AR Path="/5DB73B0A" Ref="R108"  Part="1"
 AR Path="/5C8C5FC0/5DB73B0A" Ref="R?"  Part="1"
-F 0 "R108" V 6425 3450 50  0000 C CNN
-F 1 "1k" V 6475 3300 50  0000 C CNN
-F 2 "AJ:R_0805_AJ" V 6405 3300 50  0001 C CNN
-F 3 "~" H 6475 3300 50  0001 C CNN
-	1    6475 3300
+F 0 "R108" V 6300 3200 50  0000 C CNN
+F 1 "1k" V 6350 3400 50  0000 C CNN
+F 2 "AJ:R_0805_AJ" V 6280 3400 50  0001 C CNN
+F 3 "~" H 6350 3400 50  0001 C CNN
+	1    6350 3400
 	0    1    1    0
 $EndComp
@@
 Connection ~ 5950 2550
 Wire Wire Line
-	6625 3200 7000 3200
-Wire Wire Line
 	6575 3700 6650 3700
 Wire Wire Line
@@
 Wire Wire Line
 	2300 3600 2350 3600
-Wire Wire Line
-	6625 3300 7000 3300
 $Comp
 L Diode:LL4148 D?
@@
 Wire Wire Line
 	2350 3600 2500 3600
+Wire Wire Line
+	6900 3600 6900 3400
+Wire Wire Line
+	6500 3400 6900 3400
+Wire Wire Line
+	6500 3300 7000 3300
 $EndSCHEMATC
