File: KicadJE_SympleSeq_Control.sch (KiCad schematic (older format))
At the start: 16 parts

Commit message: Annotate #1
Parts:
- removed RV? (x2): R_POT, symbol Device:R_POT
- removed RV?: R_POT, AJ:Potentiometer_China_RK09_Single_Vertical_AJ, symbol Device:R_POT
- added RV? (x3): CV4, AJ-Dropbox-Kicad:Potentiometer_China_RK09_Single_Vertical_AJ, symbol Device:R_POT
- RV304: renamed from RV?; value R_POT -> CV4; footprint (none) -> AJ-Dropbox-Kicad:Potentiometer_China_RK09_Single_Vertical_AJ
- gave numbers to parts that had none: 12
Connections:
- net CV: now also RV?.2, RV?.2, RV?.2
- net Gate: now also RV?.1, RV?.1, RV?.1
- net at R303.2: now also RV?.3
- net at R302.2: now also RV?.3
- net at R301.2: now also RV?.3
Changed lines of the file:
@@
 $EndDescr
 $Comp
-L Device:LED D?
+L Device:LED D304
 U 1 1 5D8FA8D7
 P 4500 4150
-F 0 "D?" V 4750 4150 50  0000 R CNN
+F 0 "D304" V 4750 4150 50  0000 R CNN
 F 1 "LED" V 4650 4150 50  0000 R CNN
 F 2 "LED_THT:LED_D5.0mm" H 4500 4150 50  0001 C CNN
@@
 $EndComp
 $Comp
-L Device:R_POT RV?
+L Device:R_POT RV304
 U 1 1 5D8FD9D8
 P 5000 4150
-F 0 "RV?" H 4931 4196 50  0000 R CNN
-F 1 "R_POT" H 4931 4105 50  0000 R CNN
-F 2 "" H 5000 4150 50  0001 C CNN
+F 0 "RV304" H 4930 4196 50  0000 R CNN
+F 1 "CV4" H 4930 4105 50  0000 R CNN
+F 2 "AJ-Dropbox-Kicad:Potentiometer_China_RK09_Single_Vertical_AJ" H 5000 4150 50  0001 C CNN
 F 3 "~" H 5000 4150 50  0001 C CNN
 	1    5000 4150
@@
 $EndComp
 $Comp
-L Switch:SW_SPDT SW?
+L Switch:SW_SPDT SW304
 U 1 1 5D8FE28E
 P 4300 3600
-F 0 "SW?" H 4300 3885 50  0000 C CNN
+F 0 "SW304" H 4300 3885 50  0000 C CNN
 F 1 "SW_SPDT" H 4300 3794 50  0000 C CNN
 F 2 "" H 4300 3600 50  0001 C CNN
@@
 	5000 3700 5000 4000
 $Comp
-L Device:R R?
+L Device:R R304
 U 1 1 5D900B45
 P 4500 4650
-F 0 "R?" H 4570 4696 50  0000 L CNN
+F 0 "R304" H 4570 4696 50  0000 L CNN
 F 1 "R" H 4570 4605 50  0000 L CNN
 F 2 "" V 4430 4650 50  0001 C CNN
@@
 	5300 4150 5150 4150
 $Comp
-L Device:LED D?
+L Device:LED D303
 U 1 1 5D902318
 P 2550 4100
-F 0 "D?" V 2800 4100 50  0000 R CNN
+F 0 "D303" V 2800 4100 50  0000 R CNN
 F 1 "LED" V 2700 4100 50  0000 R CNN
 F 2 "LED_THT:LED_D5.0mm" H 2550 4100 50  0001 C CNN
@@
 $EndComp
 $Comp
-L Device:R_POT RV?
-U 1 1 5D902322
-P 3050 4100
-F 0 "RV?" H 2981 4146 50  0000 R CNN
-F 1 "R_POT" H 2981 4055 50  0000 R CNN
-F 2 "" H 3050 4100 50  0001 C CNN
-F 3 "~" H 3050 4100 50  0001 C CNN
-	1    3050 4100
-	1    0    0    -1
-$EndComp
-$Comp
-L Switch:SW_SPDT SW?
+L Switch:SW_SPDT SW303
 U 1 1 5D90232C
 P 2350 3550
-F 0 "SW?" H 2350 3835 50  0000 C CNN
+F 0 "SW303" H 2350 3835 50  0000 C CNN
 F 1 "SW_SPDT" H 2350 3744 50  0000 C CNN
 F 2 "" H 2350 3550 50  0001 C CNN
@@
 	3050 3650 3050 3950
 $Comp
-L Device:R R?
+L Device:R R303
 U 1 1 5D90233A
 P 2550 4600
-F 0 "R?" H 2620 4646 50  0000 L CNN
+F 0 "R303" H 2620 4646 50  0000 L CNN
 F 1 "R" H 2620 4555 50  0000 L CNN
 F 2 "" V 2480 4600 50  0001 C CNN
@@
 	3350 4100 3200 4100
 $Comp
-L Device:LED D?
+L Device:LED D302
 U 1 1 5D90557F
 P 4500 2300
-F 0 "D?" V 4750 2300 50  0000 R CNN
+F 0 "D302" V 4750 2300 50  0000 R CNN
 F 1 "LED" V 4650 2300 50  0000 R CNN
 F 2 "LED_THT:LED_D5.0mm" H 4500 2300 50  0001 C CNN
@@
 $EndComp
 $Comp
-L Device:R_POT RV?
-U 1 1 5D905589
-P 5000 2300
-F 0 "RV?" H 4931 2346 50  0000 R CNN
-F 1 "R_POT" H 4931 2255 50  0000 R CNN
-F 2 "" H 5000 2300 50  0001 C CNN
-F 3 "~" H 5000 2300 50  0001 C CNN
-	1    5000 2300
-	1    0    0    -1
-$EndComp
-$Comp
-L Switch:SW_SPDT SW?
+L Switch:SW_SPDT SW302
 U 1 1 5D905593
 P 4300 1750
-F 0 "SW?" H 4300 2035 50  0000 C CNN
+F 0 "SW302" H 4300 2035 50  0000 C CNN
 F 1 "SW_SPDT" H 4300 1944 50  0000 C CNN
 F 2 "" H 4300 1750 50  0001 C CNN
@@
 	5000 1850 5000 2150
 $Comp
-L Device:R R?
+L Device:R R302
 U 1 1 5D9055A1
 P 4500 2800
-F 0 "R?" H 4570 2846 50  0000 L CNN
+F 0 "R302" H 4570 2846 50  0000 L CNN
 F 1 "R" H 4570 2755 50  0000 L CNN
 F 2 "" V 4430 2800 50  0001 C CNN
@@
 	5300 2300 5150 2300
 $Comp
-L Device:LED D?
+L Device:LED D301
 U 1 1 5D9055B8
 P 2550 2250
-F 0 "D?" V 2800 2250 50  0000 R CNN
+F 0 "D301" V 2800 2250 50  0000 R CNN
 F 1 "LED" V 2700 2250 50  0000 R CNN
 F 2 "LED_THT:LED_D5.0mm" H 2550 2250 50  0001 C CNN
@@
 $EndComp
 $Comp
-L Device:R_POT RV?
-U 1 1 5D9055C2
-P 3050 2250
-F 0 "RV?" H 2981 2296 50  0000 R CNN
-F 1 "R_POT" H 2981 2205 50  0000 R CNN
-F 2 "AJ:Potentiometer_China_RK09_Single_Vertical_AJ" H 3050 2250 50  0001 C CNN
-F 3 "~" H 3050 2250 50  0001 C CNN
-	1    3050 2250
-	1    0    0    -1
-$EndComp
-$Comp
-L Switch:SW_SPDT SW?
+L Switch:SW_SPDT SW301
 U 1 1 5D9055CC
 P 2350 1700
-F 0 "SW?" H 2350 1985 50  0000 C CNN
+F 0 "SW301" H 2350 1985 50  0000 C CNN
 F 1 "SW_SPDT" H 2350 1894 50  0000 C CNN
 F 2 "" H 2350 1700 50  0001 C CNN
@@
 	3050 1800 3050 2100
 $Comp
-L Device:R R?
+L Device:R R301
 U 1 1 5D9055DA
 P 2550 2750
-F 0 "R?" H 2620 2796 50  0000 L CNN
+F 0 "R301" H 2620 2796 50  0000 L CNN
 F 1 "R" H 2620 2705 50  0000 L CNN
 F 2 "" V 2480 2750 50  0001 C CNN
@@
 Wire Wire Line
 	3350 2250 3200 2250
+$Comp
+L Device:R_POT RV?
+U 1 1 5DB97621
+P 3050 4100
+F 0 "RV?" H 2980 4146 50  0000 R CNN
+F 1 "CV4" H 2980 4055 50  0000 R CNN
+F 2 "AJ-Dropbox-Kicad:Potentiometer_China_RK09_Single_Vertical_AJ" H 3050 4100 50  0001 C CNN
+F 3 "~" H 3050 4100 50  0001 C CNN
+	1    3050 4100
+	1    0    0    -1
+$EndComp
+$Comp
+L Device:R_POT RV?
+U 1 1 5DB97C6D
+P 3050 2250
+F 0 "RV?" H 2980 2296 50  0000 R CNN
+F 1 "CV4" H 2980 2205 50  0000 R CNN
+F 2 "AJ-Dropbox-Kicad:Potentiometer_China_RK09_Single_Vertical_AJ" H 3050 2250 50  0001 C CNN
+F 3 "~" H 3050 2250 50  0001 C CNN
+	1    3050 2250
+	1    0    0    -1
+$EndComp
+$Comp
+L Device:R_POT RV?
+U 1 1 5DB98203
+P 5000 2300
+F 0 "RV?" H 4930 2346 50  0000 R CNN
+F 1 "CV4" H 4930 2255 50  0000 R CNN
+F 2 "AJ-Dropbox-Kicad:Potentiometer_China_RK09_Single_Vertical_AJ" H 5000 2300 50  0001 C CNN
+F 3 "~" H 5000 2300 50  0001 C CNN
+	1    5000 2300
+	1    0    0    -1
+$EndComp
 $EndSCHEMATC

Commit message: control module PCB init
Parts:
- added D305, D306, D307, D308, D309, D310, D311, D312: LL4148, Diode_SMD:D_MiniMELF, symbol Diode:LL4148
- R301, R302, R303, R304: value R -> 12k; footprint (none) -> AJ:D_0805_2012Metric_Pad1.15x1.40mm_HandSolder
- RV301: renamed from RV?; value CV4 -> CV1
- RV302: renamed from RV?; value CV4 -> CV2
- RV303: renamed from RV?; value CV4 -> CV3
- SW301, SW302, SW303, SW304: footprint (none) -> AJ:SP1MS1
Connections:
- net CV: now also D307.1 (K), D308.1 (K), D311.1 (K), D312.1 (K); no longer RV301.2, RV302.2, RV303.2, RV304.2
- net Gate: now also D305.1 (K), D306.1 (K), D309.1 (K), D310.1 (K); no longer D301.2 (A), D302.2 (A), D303.2 (A), D304.2 (A), RV301.1, RV302.1, RV303.1, RV304.1, SW301.3 (C), SW302.3 (C), SW303.3 (C), SW304.3 (C)
- net GND: now reaches R304.2, RV304.3
- net GND: now also R301.2, R302.2, R303.2, RV301.3, RV302.3, RV303.3
- new net: D304.2 (A), D310.2 (A), RV304.1, SW304.3 (C)
- new net: D312.2 (A), RV304.2
- new net: D303.2 (A), D309.2 (A), RV303.1, SW303.3 (C)
- new net: D302.2 (A), D306.2 (A), RV302.1, SW302.3 (C)
- new net: D301.2 (A), D305.2 (A), RV301.1, SW301.3 (C)
- new net: D311.2 (A), RV303.2
- new net: D307.2 (A), RV301.2
- new net: D308.2 (A), RV302.2
