File: KicadJE_SympleSeq_Control.sch (KiCad schematic (older format))
At the start: 24 parts, among them SW301 SW_SPDT, SW302 SW_SPDT, SW303 SW_SPDT, SW304 SW_SPDT

Commit message: AJ Footprints
Parts:
- D301, D302, D303, D304: footprint LED_THT:LED_D5.0mm -> AJ:D_0805_2012Metric_Pad1.15x1.40mm_HandSolder
- R301, R302, R303, R304: footprint AJ:D_0805_2012Metric_Pad1.15x1.40mm_HandSolder -> AJ:R_0805_2012Metric_Pad1.15x1.40mm_HandSolder
Changed lines of the file:
@@
 F 0 "D304" V 4750 4150 50  0000 R CNN
 F 1 "LED" V 4650 4150 50  0000 R CNN
-F 2 "LED_THT:LED_D5.0mm" H 4500 4150 50  0001 C CNN
+F 2 "AJ:D_0805_2012Metric_Pad1.15x1.40mm_HandSolder" H 4500 4150 50  0001 C CNN
 F 3 "~" H 4500 4150 50  0001 C CNN
 	1    4500 4150
@@
 F 0 "R304" H 4570 4696 50  0000 L CNN
 F 1 "12k" H 4570 4605 50  0000 L CNN
-F 2 "AJ:D_0805_2012Metric_Pad1.15x1.40mm_HandSolder" V 4430 4650 50  0001 C CNN
+F 2 "AJ:R_0805_2012Metric_Pad1.15x1.40mm_HandSolder" V 4430 4650 50  0001 C CNN
 F 3 "~" H 4500 4650 50  0001 C CNN
 	1    4500 4650
@@
 F 0 "D303" V 2800 4100 50  0000 R CNN
 F 1 "LED" V 2700 4100 50  0000 R CNN
-F 2 "LED_THT:LED_D5.0mm" H 2550 4100 50  0001 C CNN
+F 2 "AJ:D_0805_2012Metric_Pad1.15x1.40mm_HandSolder" H 2550 4100 50  0001 C CNN
 F 3 "~" H 2550 4100 50  0001 C CNN
 	1    2550 4100
@@
 F 0 "R303" H 2620 4646 50  0000 L CNN
 F 1 "12k" H 2620 4555 50  0000 L CNN
-F 2 "AJ:D_0805_2012Metric_Pad1.15x1.40mm_HandSolder" V 2480 4600 50  0001 C CNN
+F 2 "AJ:R_0805_2012Metric_Pad1.15x1.40mm_HandSolder" V 2480 4600 50  0001 C CNN
 F 3 "~" H 2550 4600 50  0001 C CNN
 	1    2550 4600
@@
 F 0 "D302" V 4750 2300 50  0000 R CNN
 F 1 "LED" V 4650 2300 50  0000 R CNN
-F 2 "LED_THT:LED_D5.0mm" H 4500 2300 50  0001 C CNN
+F 2 "AJ:D_0805_2012Metric_Pad1.15x1.40mm_HandSolder" H 4500 2300 50  0001 C CNN
 F 3 "~" H 4500 2300 50  0001 C CNN
 	1    4500 2300
@@
 F 0 "R302" H 4570 2846 50  0000 L CNN
 F 1 "12k" H 4570 2755 50  0000 L CNN
-F 2 "AJ:D_0805_2012Metric_Pad1.15x1.40mm_HandSolder" V 4430 2800 50  0001 C CNN
+F 2 "AJ:R_0805_2012Metric_Pad1.15x1.40mm_HandSolder" V 4430 2800 50  0001 C CNN
 F 3 "~" H 4500 2800 50  0001 C CNN
 	1    4500 2800
@@
 F 0 "D301" V 2800 2250 50  0000 R CNN
 F 1 "LED" V 2700 2250 50  0000 R CNN
-F 2 "LED_THT:LED_D5.0mm" H 2550 2250 50  0001 C CNN
+F 2 "AJ:D_0805_2012Metric_Pad1.15x1.40mm_HandSolder" H 2550 2250 50  0001 C CNN
 F 3 "~" H 2550 2250 50  0001 C CNN
 	1    2550 2250
@@
 F 0 "R301" H 2620 2796 50  0000 L CNN
 F 1 "12k" H 2620 2705 50  0000 L CNN
-F 2 "AJ:D_0805_2012Metric_Pad1.15x1.40mm_HandSolder" V 2480 2750 50  0001 C CNN
+F 2 "AJ:R_0805_2012Metric_Pad1.15x1.40mm_HandSolder" V 2480 2750 50  0001 C CNN
 F 3 "~" H 2550 2750 50  0001 C CNN
 	1    2550 2750

Commit message: AJ footprints updated
Parts:
- D301, D302, D303, D304: footprint AJ:D_0805_2012Metric_Pad1.15x1.40mm_HandSolder -> AJ:D_0805_AJ
- R301, R302, R303, R304: footprint AJ:R_0805_2012Metric_Pad1.15x1.40mm_HandSolder -> AJ:R_0805_AJ
Changed lines of the file:
@@
 F 0 "D304" V 4750 4150 50  0000 R CNN
 F 1 "LED" V 4650 4150 50  0000 R CNN
-F 2 "AJ:D_0805_2012Metric_Pad1.15x1.40mm_HandSolder" H 4500 4150 50  0001 C CNN
+F 2 "AJ:D_0805_AJ" H 4500 4150 50  0001 C CNN
 F 3 "~" H 4500 4150 50  0001 C CNN
 	1    4500 4150
@@
 F 0 "R304" H 4570 4696 50  0000 L CNN
 F 1 "12k" H 4570 4605 50  0000 L CNN
-F 2 "AJ:R_0805_2012Metric_Pad1.15x1.40mm_HandSolder" V 4430 4650 50  0001 C CNN
+F 2 "AJ:R_0805_AJ" V 4430 4650 50  0001 C CNN
 F 3 "~" H 4500 4650 50  0001 C CNN
 	1    4500 4650
@@
 F 0 "D303" V 2800 4100 50  0000 R CNN
 F 1 "LED" V 2700 4100 50  0000 R CNN
-F 2 "AJ:D_0805_2012Metric_Pad1.15x1.40mm_HandSolder" H 2550 4100 50  0001 C CNN
+F 2 "AJ:D_0805_AJ" H 2550 4100 50  0001 C CNN
 F 3 "~" H 2550 4100 50  0001 C CNN
 	1    2550 4100
@@
 F 0 "R303" H 2620 4646 50  0000 L CNN
 F 1 "12k" H 2620 4555 50  0000 L CNN
-F 2 "AJ:R_0805_2012Metric_Pad1.15x1.40mm_HandSolder" V 2480 4600 50  0001 C CNN
+F 2 "AJ:R_0805_AJ" V 2480 4600 50  0001 C CNN
 F 3 "~" H 2550 4600 50  0001 C CNN
 	1    2550 4600
@@
 F 0 "D302" V 4750 2300 50  0000 R CNN
 F 1 "LED" V 4650 2300 50  0000 R CNN
-F 2 "AJ:D_0805_2012Metric_Pad1.15x1.40mm_HandSolder" H 4500 2300 50  0001 C CNN
+F 2 "AJ:D_0805_AJ" H 4500 2300 50  0001 C CNN
 F 3 "~" H 4500 2300 50  0001 C CNN
 	1    4500 2300
@@
 F 0 "R302" H 4570 2846 50  0000 L CNN
 F 1 "12k" H 4570 2755 50  0000 L CNN
-F 2 "AJ:R_0805_2012Metric_Pad1.15x1.40mm_HandSolder" V 4430 2800 50  0001 C CNN
+F 2 "AJ:R_0805_AJ" V 4430 2800 50  0001 C CNN
 F 3 "~" H 4500 2800 50  0001 C CNN
 	1    4500 2800
@@
 F 0 "D301" V 2800 2250 50  0000 R CNN
 F 1 "LED" V 2700 2250 50  0000 R CNN
-F 2 "AJ:D_0805_2012Metric_Pad1.15x1.40mm_HandSolder" H 2550 2250 50  0001 C CNN
+F 2 "AJ:D_0805_AJ" H 2550 2250 50  0001 C CNN
 F 3 "~" H 2550 2250 50  0001 C CNN
 	1    2550 2250
@@
 F 0 "R301" H 2620 2796 50  0000 L CNN
 F 1 "12k" H 2620 2705 50  0000 L CNN
-F 2 "AJ:R_0805_2012Metric_Pad1.15x1.40mm_HandSolder" V 2480 2750 50  0001 C CNN
+F 2 "AJ:R_0805_AJ" V 2480 2750 50  0001 C CNN
 F 3 "~" H 2550 2750 50  0001 C CNN
 	1    2550 2750

Commit message: Update KicadJE_SympleSeq_Control.sch
Fix LED error 0805 -> LED_THT:LED_D3.0mm
Parts:
- D301, D302, D303, D304: footprint AJ:D_0805_AJ -> LED_THT:LED_D3.0mm
Changed lines of the file:
@@
 F 0 "D304" V 4750 4150 50  0000 R CNN
 F 1 "LED" V 4650 4150 50  0000 R CNN
-F 2 "AJ:D_0805_AJ" H 4500 4150 50  0001 C CNN
+F 2 "LED_THT:LED_D3.0mm" H 4500 4150 50  0001 C CNN
 F 3 "~" H 4500 4150 50  0001 C CNN
 	1    4500 4150
@@
 F 0 "D303" V 2800 4100 50  0000 R CNN
 F 1 "LED" V 2700 4100 50  0000 R CNN
-F 2 "AJ:D_0805_AJ" H 2550 4100 50  0001 C CNN
+F 2 "LED_THT:LED_D3.0mm" H 2550 4100 50  0001 C CNN
 F 3 "~" H 2550 4100 50  0001 C CNN
 	1    2550 4100
@@
 F 0 "D302" V 4750 2300 50  0000 R CNN
 F 1 "LED" V 4650 2300 50  0000 R CNN
-F 2 "AJ:D_0805_AJ" H 4500 2300 50  0001 C CNN
+F 2 "LED_THT:LED_D3.0mm" H 4500 2300 50  0001 C CNN
 F 3 "~" H 4500 2300 50  0001 C CNN
 	1    4500 2300
@@
 F 0 "D301" V 2800 2250 50  0000 R CNN
 F 1 "LED" V 2700 2250 50  0000 R CNN
-F 2 "AJ:D_0805_AJ" H 2550 2250 50  0001 C CNN
+F 2 "LED_THT:LED_D3.0mm" H 2550 2250 50  0001 C CNN
 F 3 "~" H 2550 2250 50  0001 C CNN
 	1    2550 2250
