File: KicadJE_SympleSeq.kicad_pcb (KiCad board)
At the start: 2 copper layers, 100 x 100 mm, 28 parts, among them J201 In1.1, J202 In1.2, J203 In1.3, J204 Out1, J205 In2, J206 Out2.1, J207 Out2.2, J208 Out2.3, P201 HEADER_2x5_Doepfer, SW201 Inv/NonInv, SW202 Inv/NonInv, U201 TL082

Commit message: control module PCB init
Parts:
- removed J205: In2, AJ-Dropbox-Kicad:PJ301SM
- removed J206: Out2.1, AJ-Dropbox-Kicad:PJ301SM
- removed J207: Out2.2, AJ-Dropbox-Kicad:PJ301SM
- removed J208: Out2.3, AJ-Dropbox-Kicad:PJ301SM
- removed R212: 47k, Resistor_SMD:R_0805_2012Metric_Pad1.15x1.40mm_HandSolder
- removed R213, R214: 4k7, Resistor_SMD:R_0805_2012Metric_Pad1.15x1.40mm_HandSolder
- removed SW201, SW202: Inv/NonInv, AJ-Dropbox-Kicad:SP1MS1
- added C203: 1u, Capacitor_SMD:C_0805_2012Metric_Pad1.15x1.40mm_HandSolder, F.Cu at (256.6, 62.7)
- added C204: 1u, Capacitor_SMD:C_1206_3216Metric_Pad1.42x1.75mm_HandSolder, F.Cu at (258.5, 47.7)
- added C205: 1u, Capacitor_SMD:C_0805_2012Metric_Pad1.15x1.40mm_HandSolder, F.Cu at (260.3, 56.8)
- added C206: 1u, Capacitor_SMD:C_1206_3216Metric_Pad1.42x1.75mm_HandSolder, F.Cu at (145.0, 133.4)
- added D201: 5817, LED_SMD:LED_0805_2012Metric, F.Cu at (250.5, 71.6)
- added D202: 5817, LED_SMD:LED_0805_2012Metric, F.Cu at (255.3, 68.3)
- added D203: 5817, LED_SMD:LED_0805_2012Metric, F.Cu at (264.9, 59.8)
- added D204: 5817, LED_SMD:LED_0805_2012Metric, F.Cu at (259.7, 65.7)
- added D205: 5817, LED_SMD:LED_0805_2012Metric, F.Cu at (250.5, 74.6)
- added D206: 5817, LED_SMD:LED_0805_2012Metric, F.Cu at (255.0, 71.6)
- added D301: LED, LED_THT:LED_D5.0mm, F.Cu at (169.0, 55.6)
- added D302: LED, LED_THT:LED_D5.0mm, F.Cu at (129.0, 55.5)
- added D303: LED, LED_THT:LED_D5.0mm, F.Cu at (108.5, 55.5)
- added D304: LED, LED_THT:LED_D5.0mm, F.Cu at (148.5, 55.5)
- added D305: LL4148, Diode_SMD:D_MiniMELF, B.Cu at (137.2, 40.9)
- added D306: LL4148, Diode_SMD:D_MiniMELF, B.Cu at (137.2, 37.6)
- added D307: LL4148, Diode_SMD:D_MiniMELF, B.Cu at (143.5, 40.9)
- added D308: LL4148, Diode_SMD:D_MiniMELF, B.Cu at (137.2, 34.4)
- added D309: LL4148, Diode_SMD:D_MiniMELF, B.Cu at (143.5, 37.6)
- added D310: LL4148, Diode_SMD:D_MiniMELF, B.Cu at (156.5, 55.5)
- added D311: LL4148, Diode_SMD:D_MiniMELF, B.Cu at (143.0, 30.5)
- added D312: LL4148, Diode_SMD:D_MiniMELF, B.Cu at (149.9, 37.6)
- added J101: CV-Out, Connector_PinHeader_2.54mm:PinHeader_1x02_P2.54mm_Vertical, F.Cu at (287.3, 58.1)
- added J102: Reset + Step, Connector_PinHeader_2.54mm:PinHeader_1x06_P2.54mm_Vertical, F.Cu at (102.5, 80.0)
- added J103: CV-G8_Mod1, Connector_PinHeader_2.54mm:PinHeader_1x03_P2.54mm_Vertical, F.Cu at (102.5, 52.9)
- added J104: CV-G8_Mod2, Connector_PinHeader_2.54mm:PinHeader_1x03_P2.54mm_Vertical, F.Cu at (178.0, 53.0)
- added J105: Clk_Hold, Connector_PinHeader_2.54mm:PinHeader_1x03_P2.54mm_Vertical, F.Cu at (209.5, 109.0)
- added J106: CV-Out, Connector_PinHeader_2.54mm:PinHeader_1x02_P2.54mm_Vertical, F.Cu at (291.9, 58.1)
- added J107: Reset + Step 1-4, Connector_PinHeader_2.54mm:PinHeader_1x06_P2.54mm_Vertical, F.Cu at (183.0, 21.4)
- added J108: Reset + Step 5-8, Connector_PinHeader_2.54mm:PinHeader_1x06_P2.54mm_Vertical, F.Cu at (187.6, 21.4)
- added R101: 100k, Resistor_SMD:R_0805_2012Metric_Pad1.15x1.40mm_HandSolder, F.Cu at (301.3, 47.6)
- added R102: 47k, Resistor_SMD:R_0805_2012Metric_Pad1.15x1.40mm_HandSolder, F.Cu at (287.3, 64.5)
- added R103: 1k, Resistor_SMD:R_0805_2012Metric_Pad1.15x1.40mm_HandSolder, F.Cu at (301.3, 53.5)
- added R104: 100k, Resistor_SMD:R_0805_2012Metric_Pad1.15x1.40mm_HandSolder, F.Cu at (296.6, 60.2)
- added R105: 100k, Resistor_SMD:R_0805_2012Metric_Pad1.15x1.40mm_HandSolder, F.Cu at (296.8, 63.2)
- added R106: 47k, Resistor_SMD:R_0805_2012Metric_Pad1.15x1.40mm_HandSolder, F.Cu at (301.4, 59.4)
- added R107: 1k, Resistor_SMD:R_0805_2012Metric_Pad1.15x1.40mm_HandSolder, F.Cu at (296.6, 57.3)
- added R108: 1k, Resistor_SMD:R_0805_2012Metric_Pad1.15x1.40mm_HandSolder, F.Cu at (301.4, 56.4)
- added R109: 1k, Resistor_SMD:R_0805_2012Metric_Pad1.15x1.40mm_HandSolder, F.Cu at (292.1, 64.5)
- added R110: 100k, Resistor_SMD:R_0805_2012Metric_Pad1.15x1.40mm_HandSolder, F.Cu at (301.3, 50.5)
- added R301: 12k, AJ:D_0805_2012Metric_Pad1.15x1.40mm_HandSolder, B.Cu at (169.0, 60.8)
- added R302: 12k, AJ:D_0805_2012Metric_Pad1.15x1.40mm_HandSolder, B.Cu at (129.0, 61.0)
- added R303: 12k, AJ:D_0805_2012Metric_Pad1.15x1.40mm_HandSolder, B.Cu at (108.5, 60.5)
- added R304: 12k, AJ:D_0805_2012Metric_Pad1.15x1.40mm_HandSolder, B.Cu at (148.5, 60.5)
- added RV201: 50k Rate, Connector_JST:JST_EH_B3B-EH-A_1x03_P2.50mm_Vertical, F.Cu at (191.5, 127.0)
- added RV301: CV1, AJ-Dropbox-Kicad:Potentiometer_China_RK09_Single_Vertical_AJ, F.Cu at (102.5, 72.5)
- added RV302: CV2, AJ-Dropbox-Kicad:Potentiometer_China_RK09_Single_Vertical_AJ, F.Cu at (122.5, 72.5)
- added RV303: CV3, AJ-Dropbox-Kicad:Potentiometer_China_RK09_Single_Vertical_AJ, F.Cu at (142.5, 72.5)
- added RV304: CV4, AJ-Dropbox-Kicad:Potentiometer_China_RK09_Single_Vertical_AJ, F.Cu at (162.5, 72.5)
- added SW301: SW_SPDT, AJ:SP1MS1, F.Cu at (109.5, 89.0)
- added SW302: SW_SPDT, AJ:SP1MS1, F.Cu at (130.0, 89.0)
- added SW303: SW_SPDT, AJ:SP1MS1, F.Cu at (150.0, 89.0)
- added SW304: SW_SPDT, AJ:SP1MS1, F.Cu at (170.0, 89.0)
- added U101: TL082, AJ:AJ_SO-8_5.3x6.2mm_P1.27mm, F.Cu at (281.5, 46.5)
- added U202: 4017, AJ:SOIC-16_4.55x10.3mm_P1.27mm, F.Cu at (146.8, 125.9)
- C201: value 1u -> 22u; moved to F.Cu
- C202: value 1u -> 10n; moved to F.Cu
- J201: value In1.1 -> clk_in
- J202: value In1.2 -> clk_out
- J203: value In1.3 -> Hold
- J204: value Out1 -> Reset
- P201: moved to F.Cu
- R201: value 47k -> 3k3; moved to F.Cu
- R202: value 20k -> 220k; moved to F.Cu
- R203, R206, R208: value 47k -> 100k; moved to F.Cu
- R204: value 47k -> 10k; moved to F.Cu
- R205: value 47k -> 1k; moved to F.Cu
- R207: value 4k7 -> 10k; moved to F.Cu
- R209: value 20k -> 47k; moved to F.Cu
- R210: value 47k -> 4k7; moved to F.Cu
- R211: value 4k7 -> OPEN; moved to F.Cu
- U201: value TL082 -> LM555; moved to F.Cu
- moved R205 119.1 mm to (261.5, 53.8)
- moved R202 115.0 mm to (261.5, 50.9)
- moved C201 112.9 mm to (256.1, 53.6)
- moved C202 110.9 mm to (264.5, 47.7)
- moved R209 108.0 mm to (265.0, 56.8)
- moved R206 106.8 mm to (255.5, 59.7)
- moved R201 102.4 mm to (245.9, 71.5)
- moved R207 100.4 mm to (250.6, 68.6)
- moved R208 100.1 mm to (260.3, 59.7)
- moved R203 91.9 mm to (245.9, 68.6)
- moved R211 90.8 mm to (245.9, 74.5)
- moved R210 86.4 mm to (255.5, 56.7)
- moved R204 86.1 mm to (251.8, 65.3)
- moved U201 73.0 mm to (217.9, 72.2)
- moved J202 65.2 mm to (126.8, 135.0), turned to 0 degrees
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Connections:
- C201 pad 2: Net-(C201-Pad2) -> GND
- C202 pad 1: Net-(C201-Pad2) -> Net-(C202-Pad1)
- C202 pad 2: Net-(C202-Pad2) -> GND
- J201 pad TN: GND -> Clk555
- J202 pad TN: GND -> (no net)
- J204 pad TN: Net-(J204-PadTN) -> (no net)
- P201 pad 1: Net-(C202-Pad2) -> -12Vc
- P201 pad 10: Net-(C201-Pad1) -> +12Vc
- P201 pad 2: Net-(C202-Pad2) -> -12Vc
- P201 pad 3: Net-(C201-Pad2) -> Net-(C203-Pad2)
- P201 pad 5: Net-(C201-Pad2) -> Net-(C203-Pad2)
- P201 pad 7: Net-(C201-Pad2) -> Net-(C203-Pad2)
- P201 pad 9: Net-(C201-Pad1) -> +12Vc
- R201 pad 2: GND -> Net-(C201-Pad1)
- R202 pad 1: Out1 -> Net-(C201-Pad1)
- R202 pad 2: Net-(R201-Pad1) -> +12Vc
- R203 pad 1: In1 -> +12Vc
- R203 pad 2: Net-(J201-PadT) -> /Clock/clock_out
- R204 pad 1: In1 -> /Clock/clock_out
- R204 pad 2: Net-(J202-PadT) -> Net-(J201-PadT)
- R205 pad 1: In1 -> /Clock/clock_out
- R205 pad 2: Net-(J203-PadT) -> Net-(J202-PadT)
- R206 pad 1: GND -> +12Vc
- R206 pad 2: Net-(R206-Pad2) -> /Clock/hold
- R207 pad 1: Out1 -> /Clock/hold
- R207 pad 2: Net-(J204-PadT) -> Net-(J203-PadT)
- R208 pad 1: Net-(R208-Pad1) -> +12Vc
- R208 pad 2: GND -> /Clock/reset
- R209 pad 1: Out2 -> /Clock/reset
- R209 pad 2: Net-(R208-Pad1) -> Net-(J204-PadT)
- R210 pad 1: In2 -> /Clock/Q8
- R210 pad 2: Net-(J205-PadT) -> /Clock/reset
- R211 pad 1: Out2 -> /Clock/Q7
- R211 pad 2: Net-(J206-PadT) -> /Clock/reset
- U201 pad 1: Out1 -> GND
- U201 pad 2: Net-(R201-Pad1) -> Net-(C201-Pad1)
- U201 pad 3: Net-(R206-Pad2) -> Clk555
- U201 pad 4: Net-(C202-Pad2) -> +12Vc
- U201 pad 5: Net-(R212-Pad2) -> Net-(C202-Pad1)
- U201 pad 6: Net-(R208-Pad1) -> Net-(C201-Pad1)
- U201 pad 7: Out2 -> (no net)
- U201 pad 8: Net-(C201-Pad1) -> +12Vc
Routing:
- net /Control IO/reset: track 0.00 -> 81.8 mm
- net /Control IO/In_4: track 0.00 -> 70.2 mm
- net /Control IO/In_3: track 0.00 -> 49.1 mm
- net /Control IO/In_2: track 0.00 -> 28.8 mm
- net Net-(D304-Pad2): track 0.00 -> 15.4 mm
- net Net-(D303-Pad2): track 0.00 -> 15.4 mm
- net Net-(D302-Pad2): track 0.00 -> 15.4 mm
- net Net-(D301-Pad2): track 0.00 -> 14.7 mm
- net /Control IO/In_1: track 0.00 -> 7.48 mm
Other:
- board size 100 x 100 mm -> 80 x 100 mm
- board text added: "JE - SympleSeq Control - RevA - 2019/9/30"
- board text added: "JE SympleSeq Clock 2019/9/30"
- board text removed: "JE MMX1 2019/3/13"

Commit message: Control Done PCB
Parts:
- moved J107 128.1 mm to (88.2, 107.7)
- moved J108 128.1 mm to (92.9, 107.7)
- moved R301 60.5 mm to (108.5, 60.5)
- moved D301 60.5 mm to (108.5, 55.5)
- moved D307 44.2 mm to (110.2, 70.0), turned to 180 degrees
- moved D311 40.1 mm to (150.0, 70.0), turned to 180 degrees
- moved D303 40.0 mm to (148.5, 55.5)
- moved R303 40.0 mm to (148.5, 60.5)
- moved D312 38.1 mm to (170.0, 70.0), turned to 180 degrees
- moved D308 36.3 mm to (130.0, 70.0), turned to 180 degrees
- moved D305 31.0 mm to (113.0, 60.2), turned to 90 degrees
- moved D309 24.8 mm to (153.0, 60.5), turned to 90 degrees
- moved D306 23.3 mm to (133.0, 60.5), turned to 90 degrees
- moved D304 20.0 mm to (168.5, 55.5)
- moved R304 20.0 mm to (168.5, 60.5)
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Routing:
- net G8_M: track 0.00 -> 128.9 mm
- net CV_M: track 0.00 -> 105.0 mm
- net Net-(D304-Pad2): track 15.4 -> 41.9 mm, vias 0 -> 2
- net Net-(D302-Pad2): track 15.4 -> 41.7 mm, vias 0 -> 2
- net Net-(D303-Pad2): track 15.4 -> 41.7 mm, vias 0 -> 2
- net Net-(D301-Pad2): track 14.7 -> 40.1 mm, vias 0 -> 2
- net GND: track 0.00 -> 15.5 mm, vias 0 -> 14
- net Net-(D307-Pad2): track 0.00 -> 6.00 mm
- net Net-(D312-Pad2): track 0.00 -> 5.75 mm
- net Net-(D311-Pad2): track 0.00 -> 5.75 mm
- net Net-(D308-Pad2): track 0.00 -> 5.75 mm
- net Net-(D304-Pad1): track 0.00 -> 3.98 mm
- net Net-(D303-Pad1): track 0.00 -> 3.98 mm
- net Net-(D301-Pad1): track 0.00 -> 3.98 mm
- net Net-(D302-Pad1): track 0.00 -> 3.95 mm
- added copper zone on B.Cu, net GND
- added copper zone on F.Cu, net GND
Other:
- board text added: "CV G8 GND"
- board text added: "RST IN4 IN3 IN2 IN1 GND"
