File: KicadJE_SympleSeq.kicad_pcb (KiCad board)
At the start: 2 copper layers, 80 x 100 mm, 74 parts, among them J101 CV-Out, J102 Reset + Step, J103 CV-G8_Mod1, J104 CV-G8_Mod2, J105 Clk_Hold, J106 CV-Out, J107 Reset + Step 1-4, J108 Reset + Step 5-8, J201 clk_in, J202 clk_out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

Commit message: clock board done
Parts:
- added J109: CV-G8_Base, Connector_PinHeader_2.54mm:PinHeader_1x03_P2.54mm_Vertical, F.Cu at (176.5, 125.0)
- C202: footprint Capacitor_SMD:C_1206_3216Metric_Pad1.42x1.75mm_HandSolder -> Capacitor_SMD:C_0805_2012Metric_Pad1.15x1.40mm_HandSolder
- C204, C206: moved to B.Cu
- J106: value CV-Out -> G8-Out
- J201, J202, J203, J204: footprint AJ-Dropbox-Kicad:PJ301SM -> Connector_Audio:Jack_3.5mm_Ledino_KB3SPRS_Horizontal
- moved C202 166.0 mm to (117.0, 124.0), turned to 270 degrees
- moved R108 165.1 mm to (144.0, 106.5), turned to 90 degrees
- moved D202 161.2 mm to (107.5, 132.7), turned to 270 degrees
- moved R202 160.2 mm to (117.0, 120.0), turned to 90 degrees
- moved R101 159.1 mm to (153.5, 106.5), turned to 90 degrees
- moved C205 159.0 mm to (112.5, 115.5), turned to 180 degrees
- moved R107 156.5 mm to (148.0, 106.5), turned to 90 degrees
- moved R103 155.1 mm to (155.5, 106.5), turned to 270 degrees
- moved R204 154.7 mm to (112.5, 132.5), turned to 270 degrees
- moved D201 153.7 mm to (107.5, 128.0), turned to 270 degrees
- moved R104 153.4 mm to (153.5, 115.5), turned to 90 degrees
- moved R205 153.2 mm to (130.0, 132.5), turned to 270 degrees
- moved C201 151.7 mm to (121.5, 123.5), turned to 270 degrees
- moved R201 151.3 mm to (102.5, 120.0)
- moved R110 149.6 mm to (168.5, 119.5), turned to 270 degrees
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Connections:
- C203 pad 2: Net-(C203-Pad2) -> GND
- C204 pad 2: Net-(C203-Pad2) -> GND
- C205 pad 2: Net-(C203-Pad2) -> GND
- C206 pad 1: Net-(C203-Pad2) -> GND
- D201 pad 2: (no net) -> /Clock/clock_out
- P201 pad 3: Net-(C203-Pad2) -> GND
- P201 pad 4: Net-(P201-Pad4) -> GND
- P201 pad 5: Net-(C203-Pad2) -> GND
- P201 pad 6: Net-(P201-Pad4) -> GND
- P201 pad 7: Net-(C203-Pad2) -> GND
- P201 pad 8: Net-(P201-Pad4) -> GND
Routing:
- net +12Vc: track 0.00 -> 160.6 mm
- net /Clock/reset: track 0.00 -> 139.7 mm, vias 0 -> 2
- net GND: track 15.5 -> 124.0 mm, vias 14 -> 38
- net /Clock/clock_out: track 0.00 -> 75.4 mm, vias 0 -> 2
- net /Clock/hold: track 0.00 -> 66.0 mm, vias 0 -> 2
- net Clk555: track 0.00 -> 43.0 mm
- net G8_M: track 128.9 -> 166.9 mm
- net CV_M: track 105.0 -> 137.6 mm
- net /Clock/Q2: track 0.00 -> 31.2 mm
- net /Clock/Q4: track 0.00 -> 23.2 mm
- net /Clock/Q1: track 0.00 -> 22.9 mm
- net /Clock/Q3: track 0.00 -> 22.6 mm
- net Net-(C201-Pad1): track 0.00 -> 21.4 mm
- net -12Vc: track 0.00 -> 20.5 mm
- net /Clock/Q0: track 0.00 -> 20.1 mm
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Other:
- board text added: "*"
