File: _autosave-KicadJE_SympleSeq.kicad_pcb (KiCad board)
At the start: 2 copper layers, 80 x 100 mm, 74 parts, among them J101 CV-Out, J102 Reset + Step, J103 CV-G8_Mod1, J104 CV-G8_Mod2, J105 Clk_Hold, J106 CV-Out, J107 Reset + Step 1-4, J108 Reset + Step 5-8, J201 clk_in, J202 clk_out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

Commit message: Init Clock board
Parts:
- added REF**: MountingHole_2.2mm_M2_Pad_Via, MountingHole:MountingHole_2.2mm_M2_Pad_Via, F.Cu at (160.0, 55.0)
- added REF**: MountingHole_2.2mm_M2_Pad_Via, MountingHole:MountingHole_2.2mm_M2_Pad_Via, F.Cu at (118.3, 55.0)
- added REF**: MountingHole_2.2mm_M2_Pad_Via, MountingHole:MountingHole_2.2mm_M2_Pad_Via, F.Cu at (120.0, 93.8)
- added REF**: MountingHole_2.2mm_M2_Pad_Via, MountingHole:MountingHole_2.2mm_M2_Pad_Via, F.Cu at (160.0, 93.8)
- C206: moved to B.Cu
- moved C202 170.7 mm to (136.5, 160.7)
- moved C203 170.7 mm to (128.6, 175.7)
- moved C204 170.7 mm to (130.5, 160.7)
- moved C205 170.7 mm to (132.3, 169.8)
- moved D201 170.7 mm to (122.5, 184.6)
- moved D202 170.7 mm to (127.3, 181.3)
- moved D203 170.7 mm to (136.9, 172.8)
- moved D206 170.7 mm to (127.0, 184.6)
- moved R103 170.7 mm to (173.3, 166.5)
- moved R104 170.7 mm to (168.6, 173.2)
- moved R105 170.7 mm to (168.8, 176.2)
- moved R106 170.7 mm to (173.4, 172.4)
- moved R107 170.7 mm to (168.6, 170.3)
- moved R108 170.7 mm to (173.4, 169.4)
- moved R110 170.7 mm to (173.3, 163.5)
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Routing:
- net /Control IO/reset: track 81.8 -> 90.1 mm
