File: KicadJE_SympleSeq_Clock.sch (KiCad schematic (older format))
At the start: 0 parts

Commit message: Counter w protection
Parts:
- added C? (x2): 1u, Capacitor_SMD:C_1206_3216Metric_Pad1.42x1.75mm_HandSolder, symbol Device:C
- added C?: 10n, Capacitor_SMD:C_1206_3216Metric_Pad1.42x1.75mm_HandSolder, symbol Device:C
- added D? (x6): 5817, LED_SMD:LED_0805_2012Metric, symbol Device:LED
- added J?: clk_in, AJ-Dropbox-Kicad:PJ301SM, symbol Connector:AudioJack2_SwitchT
- added J?: clk_out, AJ-Dropbox-Kicad:PJ301SM, symbol Connector:AudioJack2_SwitchT
- added J?: Reset, AJ-Dropbox-Kicad:PJ301SM, symbol Connector:AudioJack2_SwitchT
- added J?: Hold, AJ-Dropbox-Kicad:PJ301SM, symbol Connector:AudioJack2_SwitchT
- added P?: HEADER_2x5_Doepfer, Connector_IDC:IDC-Header_2x05_P2.54mm_Vertical, symbol Eurorack:HEADER_2x5_Doepfer
- added R? (x2): 10k, Resistor_SMD:R_0805_2012Metric_Pad1.15x1.40mm_HandSolder, symbol Device:R
- added R?: 1k, Resistor_SMD:R_0805_2012Metric_Pad1.15x1.40mm_HandSolder, symbol Device:R
- added R?: 47k, Resistor_SMD:R_0805_2012Metric_Pad1.15x1.40mm_HandSolder, symbol Device:R
- added R? (x3): 100k, Resistor_SMD:R_0805_2012Metric_Pad1.15x1.40mm_HandSolder, symbol Device:R
- added R?: 4k7, Resistor_SMD:R_0805_2012Metric_Pad1.15x1.40mm_HandSolder, symbol Device:R
- added R?: OPEN, Resistor_SMD:R_0805_2012Metric_Pad1.15x1.40mm_HandSolder, symbol Device:R
- added U?: LM555, symbol Timer:LM555
- added U?: 4017, symbol 4xxx:4017
- added U?: TL082, symbol Amplifier_Operational:TL082
Connections:
- new net: C?.2, U?.1 (GND)
- new net: C?.1, U?.5 (CV)
- new net: C?.1, C?.2, P?.3 (GND), P?.5 (GND), P?.7 (GND)
- new net: P?.4 (GND), P?.6 (GND), P?.8 (GND)
- new net: J?.T, R?.2 (x4)
- new net +12Vc: C?.1, D?.1 (K), D?.1 (K), D?.1 (K), P?.10 (+12), P?.9 (+12), R?.1, R?.1, R?.1, U?.16 (VDD), U?.8 (V+)
- new net -12Vc: C?.2, P?.1 (-12), P?.2 (-12), U?.4 (V-)
- new net Carry: U?.12 (Cout)
- new net Clk555: J?.TN
- new net GND: D?.2 (A), D?.2 (A), D?.2 (A), J?.S, J?.S, J?.S, J?.S, J?.TN, U?.8 (VSS)
- new net Q0: U?.3 (Q0)
- new net Q1: U?.2 (Q1)
- new net Q2: U?.4 (Q2)
- new net Q3: U?.7 (Q3)
- new net Q4: U?.10 (Q4)
- new net Q5: U?.1 (Q5)
- new net Q6: U?.5 (Q6)
- new net Q7: R?.1, U?.6 (Q7)
- new net Q8: R?.1, U?.9 (Q8)
- new net Q9: U?.11 (Q9)
- new net clock_out: D?.1 (K), R?.1, R?.1, R?.2, U?.14 (CLK)
- new net hold: D?.1 (K), D?.2 (A), R?.1, R?.2, U?.13 (CKEN)
- new net reset: D?.1 (K), D?.2 (A), R?.1, R?.2, R?.2, R?.2, U?.15 (Reset)

Commit message: 555 done sch
Parts:
- added C?: 22u, Capacitor_SMD:C_1206_3216Metric_Pad1.42x1.75mm_HandSolder, symbol Device:C
- added C? (x2): 1u, Capacitor_SMD:C_0805_2012Metric_Pad1.15x1.40mm_HandSolder, symbol Device:C
- added R?: 220k, Resistor_SMD:R_0805_2012Metric_Pad1.15x1.40mm_HandSolder, symbol Device:R
- added R?: 3k3, Resistor_SMD:R_0805_2012Metric_Pad1.15x1.40mm_HandSolder, symbol Device:R
- added RV?: 50k, symbol Device:R_POT
- U?: footprint (none) -> AJ-Dropbox-Kicad:AJ_SO-8_5.3x6.2mm_P1.27mm
- U?: footprint (none) -> AJ:SOIC-16_4.55x10.3mm_P1.27mm
Connections:
- net +12Vc: now also U?.4 (R), U?.8 (VCC), C?.1, C?.1, R?.2
- net Clk555: now also U?.3 (Q), RV?.2, RV?.3
- net GND: now also C?.2, U?.1 (GND), C?.2
- net at U?.2 (TR): now also U?.6 (THR), C?.1, R?.1, R?.2
- net at C?.1, C?.2, P?.3 (GND)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: now also C?.2, C?.2
- new net: R?.1, RV?.1
Other:
- moved on the sheet: C?, U?, U?C
Changed lines of the file:
@@
 L Timer:LM555 U?
 U 1 1 5D9A0E3B
-P 3300 1850
+P 3350 1900
 AR Path="/5C8BFBBC/5D9A0E3B" Ref="U?"  Part="1"
 AR Path="/5D9A0E3B" Ref="U?"  Part="1"
 AR Path="/5C8C5FC0/5D9A0E3B" Ref="U?"  Part="1"
-F 0 "U?" H 3300 2428 50  0000 C CNN
-F 1 "LM555" H 3300 2337 50  0000 C CNN
-F 2 "" H 3300 1850 50  0001 C CNN
-F 3 "http://www.ti.com/lit/ds/symlink/lm555.pdf" H 3300 1850 50  0001 C CNN
-	1    3300 1850
+F 0 "U?" H 3350 2478 50  0000 C CNN
+F 1 "LM555" H 3350 2387 50  0000 C CNN
+F 2 "AJ-Dropbox-Kicad:AJ_SO-8_5.3x6.2mm_P1.27mm" H 3350 1900 50  0001 C CNN
+F 3 "http://www.ti.com/lit/ds/symlink/lm555.pdf" H 3350 1900 50  0001 C CNN
+	1    3350 1900
 	1    0    0    -1
 $EndComp
@@
 F 0 "U?" H 3350 5081 50  0000 C CNN
 F 1 "4017" H 3350 4990 50  0000 C CNN
-F 2 "" H 3350 4100 50  0001 C CNN
+F 2 "AJ:SOIC-16_4.55x10.3mm_P1.27mm" H 3350 4100 50  0001 C CNN
 F 3 "http://www.intersil.com/content/dam/Intersil/documents/cd40/cd4017bms-22bms.pdf" H 3350 4100 50  0001 C CNN
 	1    3350 4100
@@
 L Amplifier_Operational:TL082 U?
 U 3 1 5D9A0E47
-P 7850 2600
+P 8500 2600
 AR Path="/5D9A0E47" Ref="U?"  Part="3"
 AR Path="/5C8C5FC0/5D9A0E47" Ref="U?"  Part="3"
-F 0 "U?" H 7808 2646 50  0000 L CNN
-F 1 "TL082" H 7808 2555 50  0000 L CNN
-F 2 "" H 7850 2600 50  0001 C CNN
-F 3 "http://www.ti.com/lit/ds/symlink/tl081.pdf" H 7850 2600 50  0001 C CNN
-	3    7850 2600
+F 0 "U?" H 8458 2646 50  0000 L CNN
+F 1 "TL082" H 8458 2555 50  0000 L CNN
+F 2 "" H 8500 2600 50  0001 C CNN
+F 3 "http://www.ti.com/lit/ds/symlink/tl081.pdf" H 8500 2600 50  0001 C CNN
+	3    8500 2600
 	1    0    0    -1
 $EndComp
@@
 F 0 "P?" H 6700 2102 40  0000 C CNN
 F 1 "HEADER_2x5_Doepfer" H 6700 2178 40  0000 C CNN
-F 2 "Connector_IDC:IDC-Header_2x05_P2.54mm_Vertical" H 6700 2269 60  0000 C CNN
+F 2 "Connector_IDC:IDC-Header_2x05_P2.54mm_Vertical" H 6700 2000 60  0000 C CNN
 F 3 "" H 6700 2600 60  0000 C CNN
 	1    6700 2600
@@
 	6450 2200 6850 2200
 Wire Wire Line
-	7750 2200 7750 2300
+	8400 2200 8400 2300
 Wire Wire Line
 	6550 2800 6450 2800
@@
 	6450 3000 6850 3000
 Wire Wire Line
-	7750 3000 7750 2900
+	8400 3000 8400 2900
 Wire Wire Line
 	6550 2700 6550 2600
@@
 Connection ~ 6850 2200
 Wire Wire Line
-	6850 2200 7350 2200
+	6850 2200 7050 2200
 Wire Wire Line
 	6850 2800 6850 3000
@@
 $EndComp
 Wire Wire Line
-	6850 2600 7350 2600
+	6850 2600 7050 2600
 Wire Wire Line
 	7350 2600 7350 2550
@@
 Wire Wire Line
 	7350 2950 7350 3000
-Connection ~ 7350 3000
-Wire Wire Line
-	7350 3000 7750 3000
 Wire Wire Line
 	7350 2250 7350 2200
-Connection ~ 7350 2200
-Wire Wire Line
-	7350 2200 7750 2200
 Text HLabel 1850 4850 3    50   Input ~ 0
 reset
@@
 Wire Wire Line
 	1550 4400 1650 4400
-Text GLabel 7750 2200 1    50   Input ~ 0
+Text GLabel 8400 2200 1    50   Input ~ 0
 +12Vc
-Text GLabel 7750 3000 3    50   Input ~ 0
+Text GLabel 8400 3000 3    50   Input ~ 0
 -12Vc
 Text GLabel 2100 4150 2    50   Input ~ 0
@@
 L Device:C C?
 U 1 1 5D9CE9B4
-P 2500 2000
-F 0 "C?" H 2615 2046 50  0000 L CNN
-F 1 "10n" H 2615 1955 50  0000 L CNN
-F 2 "Capacitor_SMD:C_1206_3216Metric_Pad1.42x1.75mm_HandSolder" H 2538 1850 50  0001 C CNN
-F 3 "~" H 2500 2000 50  0001 C CNN
-	1    2500 2000
-	1    0    0    -1
-$EndComp
-Wire Wire Line
-	2800 1850 2500 1850
-Wire Wire Line
-	2500 2150 2500 2350
-Wire Wire Line
-	2500 2350 3300 2350
-Wire Wire Line
-	3300 2350 3300 2250
+P 2550 2050
+F 0 "C?" H 2665 2096 50  0000 L CNN
+F 1 "10n" H 2665 2005 50  0000 L CNN
+F 2 "Capacitor_SMD:C_1206_3216Metric_Pad1.42x1.75mm_HandSolder" H 2588 1900 50  0001 C CNN
+F 3 "~" H 2550 2050 50  0001 C CNN
+	1    2550 2050
+	1    0    0    -1
+$EndComp
+Wire Wire Line
+	2850 1900 2550 1900
+Wire Wire Line
+	2550 2200 2550 2400
+Wire Wire Line
+	2550 2400 3350 2400
+Wire Wire Line
+	3350 2400 3350 2300
 Wire Wire Line
 	2600 5150 2500 5150
@@
 	1250 4300 1150 4300
 Connection ~ 1150 4300
+Text GLabel 3350 1000 1    50   Input ~ 0
++12Vc
+Wire Wire Line
+	2850 2100 2800 2100
+$Comp
+L Device:C C?
+U 1 1 5DA2BD1C
+P 2150 2050
+F 0 "C?" H 2265 2096 50  0000 L CNN
+F 1 "22u" H 2265 2005 50  0000 L CNN
+F 2 "Capacitor_SMD:C_1206_3216Metric_Pad1.42x1.75mm_HandSolder" H 2188 1900 50  0001 C CNN
+F 3 "~" H 2150 2050 50  0001 C CNN
+	1    2150 2050
+	1    0    0    -1
+$EndComp
+Wire Wire Line
+	2150 1900 2150 1700
+Wire Wire Line
+	2150 1700 2550 1700
+Wire Wire Line
+	2150 2200 2150 2400
+Wire Wire Line
+	2150 2400 2550 2400
+Connection ~ 2550 2400
+$Comp
+L Device:R R?
+U 1 1 5DA35A0E
+P 2150 1450
+AR Path="/5DA35A0E" Ref="R?"  Part="1"
+AR Path="/5C8C5FC0/5DA35A0E" Ref="R?"  Part="1"
+F 0 "R?" V 2150 1450 50  0000 C CNN
+F 1 "220k" V 2034 1450 50  0000 C CNN
+F 2 "Resistor_SMD:R_0805_2012Metric_Pad1.15x1.40mm_HandSolder" V 2080 1450 50  0001 C CNN
+F 3 "~" H 2150 1450 50  0001 C CNN
+	1    2150 1450
+	-1   0    0    1
+$EndComp
+Wire Wire Line
+	3350 1000 3350 1200
+Wire Wire Line
+	2150 1300 2150 1200
+Wire Wire Line
+	2150 1200 2800 1200
+Connection ~ 3350 1200
+Wire Wire Line
+	3350 1200 3350 1500
+Wire Wire Line
+	2800 1200 2800 2100
+Connection ~ 2800 1200
+Wire Wire Line
+	2800 1200 3350 1200
+Wire Wire Line
+	2150 1600 2150 1700
+Connection ~ 2150 1700
+$Comp
+L Envelope-cache-2018-08-04-13-00-04:GND #PWR?
+U 1 1 5DA5466A
+P 3350 2400
+AR Path="/5DA5466A" Ref="#PWR?"  Part="1"
+AR Path="/5C8C5FC0/5DA5466A" Ref="#PWR?"  Part="1"
+F 0 "#PWR?" H 3350 2150 50  0001 C CNN
+F 1 "GND" H 3355 2227 50  0000 C CNN
+F 2 "" H 3350 2400 50  0001 C CNN
+F 3 "" H 3350 2400 50  0001 C CNN
+	1    3350 2400
+	1    0    0    -1
+$EndComp
+Connection ~ 3350 2400
+$Comp
+L Device:R R?
+U 1 1 5DA5509F
+P 4150 1150
+AR Path="/5DA5509F" Ref="R?"  Part="1"
+AR Path="/5C8C5FC0/5DA5509F" Ref="R?"  Part="1"
+F 0 "R?" V 4150 1100 50  0000 C CNN
+F 1 "3k3" V 4034 1150 50  0000 C CNN
+F 2 "Resistor_SMD:R_0805_2012Metric_Pad1.15x1.40mm_HandSolder" V 4080 1150 50  0001 C CNN
+F 3 "~" H 4150 1150 50  0001 C CNN
+	1    4150 1150
+	0    1    1    0
+$EndComp
+Connection ~ 2550 1700
+Wire Wire Line
+	2550 1700 2850 1700
+Text GLabel 4550 1700 2    50   Input ~ 0
+Clk555
+$Comp
+L Device:R_POT RV?
+U 1 1 5DA56D25
+P 4350 1500
+AR Path="/5C8BFBBC/5DA56D25" Ref="RV?"  Part="1"
+AR Path="/5C8C5FC0/5DA56D25" Ref="RV?"  Part="1"
+F 0 "RV?" V 4235 1500 50  0000 C CNN
+F 1 "50k" V 4144 1500 50  0000 C CNN
+F 2 "" H 4350 1500 50  0001 C CNN
+F 3 "~" H 4350 1500 50  0001 C CNN
+	1    4350 1500
+	1    0    0    -1
+$EndComp
+Wire Wire Line
+	4500 1500 4500 1700
+Wire Wire Line
+	3850 1700 4350 1700
+Wire Wire Line
+	4350 1650 4350 1700
+Connection ~ 4350 1700
+Wire Wire Line
+	4350 1700 4500 1700
+Wire Wire Line
+	4350 1150 4300 1150
+Wire Wire Line
+	4350 1150 4350 1350
+Wire Wire Line
+	4000 1150 3900 1150
+Wire Wire Line
+	2550 1150 2550 1700
+Wire Wire Line
+	3850 2100 3900 2100
+Wire Wire Line
+	3900 2100 3900 1150
+Connection ~ 3900 1150
+Wire Wire Line
+	3900 1150 2550 1150
+Wire Wire Line
+	4550 1700 4500 1700
+Connection ~ 4500 1700
+$Comp
+L Device:C C?
+U 1 1 5DAB41E4
+P 7050 2400
+F 0 "C?" H 7165 2446 50  0000 L CNN
+F 1 "1u" H 7165 2355 50  0000 L CNN
+F 2 "Capacitor_SMD:C_0805_2012Metric_Pad1.15x1.40mm_HandSolder" H 7088 2250 50  0001 C CNN
+F 3 "~" H 7050 2400 50  0001 C CNN
+	1    7050 2400
+	1    0    0    -1
+$EndComp
+Wire Wire Line
+	7050 2250 7050 2200
+Connection ~ 7050 2200
+Wire Wire Line
+	7050 2200 7350 2200
+Wire Wire Line
+	7050 2550 7050 2600
+Connection ~ 7050 2600
+Wire Wire Line
+	7050 2600 7350 2600
+Wire Wire Line
+	7350 2200 7650 2200
+Connection ~ 7350 2200
+Wire Wire Line
+	7350 3000 8400 3000
+Connection ~ 7350 3000
+$Comp
+L Device:C C?
+U 1 1 5DAD99E3
+P 7650 2400
+F 0 "C?" H 7765 2446 50  0000 L CNN
+F 1 "1u" H 7765 2355 50  0000 L CNN
+F 2 "Capacitor_SMD:C_0805_2012Metric_Pad1.15x1.40mm_HandSolder" H 7688 2250 50  0001 C CNN
+F 3 "~" H 7650 2400 50  0001 C CNN
+	1    7650 2400
+	1    0    0    -1
+$EndComp
+Wire Wire Line
+	7650 2250 7650 2200
+Connection ~ 7650 2200
+Wire Wire Line
+	7650 2200 8400 2200
+Wire Wire Line
+	7650 2550 7650 2600
+Wire Wire Line
+	7650 2600 7350 2600
 $EndSCHEMATC

Commit message: base circuit done
Changed lines of the file:
@@
 Wire Wire Line
 	7350 2250 7350 2200
-Text HLabel 1850 4850 3    50   Input ~ 0
+Text HLabel 2600 3900 3    50   Input ~ 0
 reset
-Text HLabel 1850 3950 1    50   Input ~ 0
+Text HLabel 2200 3600 3    50   Input ~ 0
 clock_out
 $Comp
@@
 AR Path="/5C8C5FC0/5D9AC299" Ref="R?"  Part="1"
 F 0 "R?" V 1400 4400 50  0000 C CNN
-F 1 "10k" V 1284 4400 50  0000 C CNN
+F 1 "10k" V 1500 4400 50  0000 C CNN
 F 2 "Resistor_SMD:R_0805_2012Metric_Pad1.15x1.40mm_HandSolder" V 1330 4400 50  0001 C CNN
 F 3 "~" H 1400 4400 50  0001 C CNN
@@
 Wire Wire Line
 	1650 4400 2250 4400
-Text HLabel 1850 4400 3    50   Input ~ 0
+Text HLabel 2350 3700 3    50   Input ~ 0
 hold
 Text HLabel 4000 3600 2    50   Input ~ 0
@@
 AR Path="/5C8C5FC0/5D9D76C7" Ref="R?"  Part="1"
 F 0 "R?" V 1850 4550 50  0000 C CNN
-F 1 "100k" V 1734 4600 50  0000 C CNN
+F 1 "100k" V 1750 4700 50  0000 C CNN
 F 2 "Resistor_SMD:R_0805_2012Metric_Pad1.15x1.40mm_HandSolder" V 1780 4600 50  0001 C CNN
 F 3 "~" H 1850 4600 50  0001 C CNN

Commit message: Annotate #1
Parts:
- RV201: renamed from RV?; value 50k -> 50k Rate; footprint (none) -> Connector_JST:JST_EH_B3B-EH-A_1x03_P2.50mm_Vertical
- gave numbers to parts that had none: 31

Commit message: control module PCB init
Parts:
- removed U101: TL082, symbol Amplifier_Operational:TL082
Changed lines of the file:
@@
-$EndComp
-$Comp
-L Amplifier_Operational:TL082 U?
-U 3 1 5D9A0E47
-P 8500 2600
-AR Path="/5D9A0E47" Ref="U?"  Part="3"
-AR Path="/5C8C5FC0/5D9A0E47" Ref="U101"  Part="3"
-F 0 "U101" H 8458 2646 50  0000 L CNN
-F 1 "TL082" H 8458 2555 50  0000 L CNN
-F 2 "" H 8500 2600 50  0001 C CNN
-F 3 "http://www.ti.com/lit/ds/symlink/tl081.pdf" H 8500 2600 50  0001 C CNN
-	3    8500 2600
-	1    0    0    -1
 $EndComp
 $Comp
@@
 	6450 2200 6850 2200
 Wire Wire Line
-	8400 2200 8400 2300
-Wire Wire Line
 	6550 2800 6450 2800
 Wire Wire Line
@@
 	6450 3000 6850 3000
 Wire Wire Line
-	8400 3000 8400 2900
-Wire Wire Line
 	6550 2700 6550 2600

Commit message: Init Clock board
Parts:
- C202: footprint Capacitor_SMD:C_1206_3216Metric_Pad1.42x1.75mm_HandSolder -> Capacitor_SMD:C_0805_2012Metric_Pad1.15x1.40mm_HandSolder
Changed lines of the file:
@@
 F 0 "C202" H 2665 2096 50  0000 L CNN
 F 1 "10n" H 2665 2005 50  0000 L CNN
-F 2 "Capacitor_SMD:C_1206_3216Metric_Pad1.42x1.75mm_HandSolder" H 2588 1900 50  0001 C CNN
+F 2 "Capacitor_SMD:C_0805_2012Metric_Pad1.15x1.40mm_HandSolder" H 2588 1900 50  0001 C CNN
 F 3 "~" H 2550 2050 50  0001 C CNN
 	1    2550 2050

Commit message: clock board done
Parts:
- J201, J202, J203, J204: footprint AJ-Dropbox-Kicad:PJ301SM -> Connector_Audio:Jack_3.5mm_Ledino_KB3SPRS_Horizontal
Connections:
- net GND: now also C203.2, C204.2, C205.2, C206.1, P201.3 (GND), P201.4 (GND), P201.5 (GND), P201.6 (GND), P201.7 (GND), P201.8 (GND)
- net clock_out: now also D201.2 (A)
Changed lines of the file:
@@
 F 0 "J201" H 830 3875 50  0000 C CNN
 F 1 "clk_in" H 600 3600 50  0000 C CNN
-F 2 "AJ-Dropbox-Kicad:PJ301SM" H 800 3550 50  0001 C CNN
+F 2 "Connector_Audio:Jack_3.5mm_Ledino_KB3SPRS_Horizontal" H 800 3550 50  0001 C CNN
 F 3 "~" H 800 3550 50  0001 C CNN
 	1    800  3550
@@
 F 0 "J202" H 830 4275 50  0000 C CNN
 F 1 "clk_out" H 600 4050 50  0000 C CNN
-F 2 "AJ-Dropbox-Kicad:PJ301SM" H 800 3950 50  0001 C CNN
+F 2 "Connector_Audio:Jack_3.5mm_Ledino_KB3SPRS_Horizontal" H 800 3950 50  0001 C CNN
 F 3 "~" H 800 3950 50  0001 C CNN
 	1    800  3950
@@
 F 0 "J204" H 830 5175 50  0000 C CNN
 F 1 "Reset" H 550 4900 50  0000 C CNN
-F 2 "AJ-Dropbox-Kicad:PJ301SM" H 800 4850 50  0001 C CNN
+F 2 "Connector_Audio:Jack_3.5mm_Ledino_KB3SPRS_Horizontal" H 800 4850 50  0001 C CNN
 F 3 "~" H 800 4850 50  0001 C CNN
 	1    800  4850
@@
 F 0 "J203" H 830 4725 50  0000 C CNN
 F 1 "Hold" H 600 4500 50  0000 C CNN
-F 2 "AJ-Dropbox-Kicad:PJ301SM" H 800 4400 50  0001 C CNN
+F 2 "Connector_Audio:Jack_3.5mm_Ledino_KB3SPRS_Horizontal" H 800 4400 50  0001 C CNN
 F 3 "~" H 800 4400 50  0001 C CNN
 	1    800  4400
@@
 	2150 3350 2100 3350
 Wire Wire Line
-	2100 3350 2100 3600
+	2100 3350 2100 3500
 Connection ~ 2100 3600
 Text GLabel 2100 4600 2    50   Input ~ 0
@@
 Wire Wire Line
 	2500 3500 2500 3350
-Wire Wire Line
-	2150 3500 2100 3500
 $Comp
 L Device:LED D?
@@
 Wire Wire Line
 	7650 2600 7350 2600
+$Comp
+L Envelope-cache-2018-08-04-13-00-04:GND #PWR?
+U 1 1 5DC0A5A8
+P 7050 2600
+AR Path="/5DC0A5A8" Ref="#PWR?"  Part="1"
+AR Path="/5C8C5FC0/5DC0A5A8" Ref="#PWR0115"  Part="1"
+F 0 "#PWR0115" H 7050 2350 50  0001 C CNN
+F 1 "GND" H 7055 2427 50  0000 C CNN
+F 2 "" H 7050 2600 50  0001 C CNN
+F 3 "" H 7050 2600 50  0001 C CNN
+	1    7050 2600
+	1    0    0    -1
+$EndComp
+$Comp
+L Envelope-cache-2018-08-04-13-00-04:GND #PWR?
+U 1 1 5DC0B21E
+P 6450 2600
+AR Path="/5DC0B21E" Ref="#PWR?"  Part="1"
+AR Path="/5C8C5FC0/5DC0B21E" Ref="#PWR0116"  Part="1"
+F 0 "#PWR0116" H 6450 2350 50  0001 C CNN
+F 1 "GND" H 6455 2427 50  0000 C CNN
+F 2 "" H 6450 2600 50  0001 C CNN
+F 3 "" H 6450 2600 50  0001 C CNN
+	1    6450 2600
+	1    0    0    -1
+$EndComp
+Wire Wire Line
+	6450 2600 6550 2600
+Wire Wire Line
+	2150 3500 2100 3500
+Connection ~ 2100 3500
+Wire Wire Line
+	2100 3500 2100 3600
 $EndSCHEMATC
