File: KicadJE_SympleSeq_Clock.sch (KiCad schematic (older format))
At the start: 40 parts, among them J201 clk_in, J202 clk_out, J203 Hold, J204 Reset, J205 Slave clock sel, P201 HEADER_2x5_Doepfer, U201 LM555, U202 4017

Commit message: AJ Footprints
Parts:
- C202, C203, C205, C207: footprint Capacitor_SMD:C_0805_2012Metric_Pad1.15x1.40mm_HandSolder -> AJ:C_0805_2012Metric_Pad1.15x1.40mm_HandSolder
- D207: footprint LED_SMD:LED_0805_2012Metric -> AJ:D_0805_2012Metric_Pad1.15x1.40mm_HandSolder
- R201, R202, R203, R204, R205, R206, R207, R208, R209, R210, R211, R212, R213, R214, R215: footprint Resistor_SMD:R_0805_2012Metric_Pad1.15x1.40mm_HandSolder -> AJ:R_0805_2012Metric_Pad1.15x1.40mm_HandSolder
Changed lines of the file:
@@
 F 0 "R204" V 1400 3550 50  0000 C CNN
 F 1 "10k" V 1284 3550 50  0000 C CNN
-F 2 "Resistor_SMD:R_0805_2012Metric_Pad1.15x1.40mm_HandSolder" V 1330 3550 50  0001 C CNN
+F 2 "AJ:R_0805_2012Metric_Pad1.15x1.40mm_HandSolder" V 1330 3550 50  0001 C CNN
 F 3 "~" H 1400 3550 50  0001 C CNN
 	1    1400 3550
@@
 F 0 "R205" V 1400 3950 50  0000 C CNN
 F 1 "1k" V 1500 3950 50  0000 C CNN
-F 2 "Resistor_SMD:R_0805_2012Metric_Pad1.15x1.40mm_HandSolder" V 1330 3950 50  0001 C CNN
+F 2 "AJ:R_0805_2012Metric_Pad1.15x1.40mm_HandSolder" V 1330 3950 50  0001 C CNN
 F 3 "~" H 1400 3950 50  0001 C CNN
 	1    1400 3950
@@
 F 0 "R207" V 1400 4400 50  0000 C CNN
 F 1 "10k" V 1500 4400 50  0000 C CNN
-F 2 "Resistor_SMD:R_0805_2012Metric_Pad1.15x1.40mm_HandSolder" V 1330 4400 50  0001 C CNN
+F 2 "AJ:R_0805_2012Metric_Pad1.15x1.40mm_HandSolder" V 1330 4400 50  0001 C CNN
 F 3 "~" H 1400 4400 50  0001 C CNN
 	1    1400 4400
@@
 F 0 "R209" V 1400 4850 50  0000 C CNN
 F 1 "47k" V 1284 4850 50  0000 C CNN
-F 2 "Resistor_SMD:R_0805_2012Metric_Pad1.15x1.40mm_HandSolder" V 1330 4850 50  0001 C CNN
+F 2 "AJ:R_0805_2012Metric_Pad1.15x1.40mm_HandSolder" V 1330 4850 50  0001 C CNN
 F 3 "~" H 1400 4850 50  0001 C CNN
 	1    1400 4850
@@
 F 0 "R206" V 1800 4150 50  0000 C CNN
 F 1 "100k" V 1684 4200 50  0000 C CNN
-F 2 "Resistor_SMD:R_0805_2012Metric_Pad1.15x1.40mm_HandSolder" V 1730 4200 50  0001 C CNN
+F 2 "AJ:R_0805_2012Metric_Pad1.15x1.40mm_HandSolder" V 1730 4200 50  0001 C CNN
 F 3 "~" H 1800 4200 50  0001 C CNN
 	1    1800 4200
@@
 F 0 "R210" V 2950 4800 50  0000 C CNN
 F 1 "4k7" V 2834 4850 50  0000 C CNN
-F 2 "Resistor_SMD:R_0805_2012Metric_Pad1.15x1.40mm_HandSolder" V 2880 4850 50  0001 C CNN
+F 2 "AJ:R_0805_2012Metric_Pad1.15x1.40mm_HandSolder" V 2880 4850 50  0001 C CNN
 F 3 "~" H 2950 4850 50  0001 C CNN
 	1    2950 4850
@@
 F 0 "R211" V 2950 5100 50  0000 C CNN
 F 1 "OPEN" V 2834 5150 50  0000 C CNN
-F 2 "Resistor_SMD:R_0805_2012Metric_Pad1.15x1.40mm_HandSolder" V 2880 5150 50  0001 C CNN
+F 2 "AJ:R_0805_2012Metric_Pad1.15x1.40mm_HandSolder" V 2880 5150 50  0001 C CNN
 F 3 "~" H 2950 5150 50  0001 C CNN
 	1    2950 5150
@@
 F 0 "C202" H 2665 2096 50  0000 L CNN
 F 1 "10n" H 2665 2005 50  0000 L CNN
-F 2 "Capacitor_SMD:C_0805_2012Metric_Pad1.15x1.40mm_HandSolder" H 2588 1900 50  0001 C CNN
+F 2 "AJ:C_0805_2012Metric_Pad1.15x1.40mm_HandSolder" H 2588 1900 50  0001 C CNN
 F 3 "~" H 2550 2050 50  0001 C CNN
 	1    2550 2050
@@
 F 0 "R203" V 1650 3300 50  0000 C CNN
 F 1 "100k" V 1534 3350 50  0000 C CNN
-F 2 "Resistor_SMD:R_0805_2012Metric_Pad1.15x1.40mm_HandSolder" V 1580 3350 50  0001 C CNN
+F 2 "AJ:R_0805_2012Metric_Pad1.15x1.40mm_HandSolder" V 1580 3350 50  0001 C CNN
 F 3 "~" H 1650 3350 50  0001 C CNN
 	1    1650 3350
@@
 F 0 "R208" V 1850 5000 50  0000 C CNN
 F 1 "100k" V 1750 5150 50  0000 C CNN
-F 2 "Resistor_SMD:R_0805_2012Metric_Pad1.15x1.40mm_HandSolder" V 1780 5050 50  0001 C CNN
+F 2 "AJ:R_0805_2012Metric_Pad1.15x1.40mm_HandSolder" V 1780 5050 50  0001 C CNN
 F 3 "~" H 1850 5050 50  0001 C CNN
 	1    1850 5050
@@
 F 0 "R202" V 2150 1450 50  0000 C CNN
 F 1 "220k" V 2034 1450 50  0000 C CNN
-F 2 "Resistor_SMD:R_0805_2012Metric_Pad1.15x1.40mm_HandSolder" V 2080 1450 50  0001 C CNN
+F 2 "AJ:R_0805_2012Metric_Pad1.15x1.40mm_HandSolder" V 2080 1450 50  0001 C CNN
 F 3 "~" H 2150 1450 50  0001 C CNN
 	1    2150 1450
@@
 F 0 "R201" V 4150 1100 50  0000 C CNN
 F 1 "3k3" V 4034 1150 50  0000 C CNN
-F 2 "Resistor_SMD:R_0805_2012Metric_Pad1.15x1.40mm_HandSolder" V 4080 1150 50  0001 C CNN
+F 2 "AJ:R_0805_2012Metric_Pad1.15x1.40mm_HandSolder" V 4080 1150 50  0001 C CNN
 F 3 "~" H 4150 1150 50  0001 C CNN
 	1    4150 1150
@@
 F 0 "C203" H 7465 2446 50  0000 L CNN
 F 1 "1u" H 7465 2355 50  0000 L CNN
-F 2 "Capacitor_SMD:C_0805_2012Metric_Pad1.15x1.40mm_HandSolder" H 7388 2250 50  0001 C CNN
+F 2 "AJ:C_0805_2012Metric_Pad1.15x1.40mm_HandSolder" H 7388 2250 50  0001 C CNN
 F 3 "~" H 7350 2400 50  0001 C CNN
 	1    7350 2400
@@
 F 0 "C205" H 8065 2446 50  0000 L CNN
 F 1 "1u" H 8065 2355 50  0000 L CNN
-F 2 "Capacitor_SMD:C_0805_2012Metric_Pad1.15x1.40mm_HandSolder" H 7988 2250 50  0001 C CNN
+F 2 "AJ:C_0805_2012Metric_Pad1.15x1.40mm_HandSolder" H 7988 2250 50  0001 C CNN
 F 3 "~" H 7950 2400 50  0001 C CNN
 	1    7950 2400
@@
 F 0 "R214" V 7100 2150 50  0000 C CNN
 F 1 "10R" V 6984 2200 50  0000 C CNN
-F 2 "Resistor_SMD:R_0805_2012Metric_Pad1.15x1.40mm_HandSolder" V 7030 2200 50  0001 C CNN
+F 2 "AJ:R_0805_2012Metric_Pad1.15x1.40mm_HandSolder" V 7030 2200 50  0001 C CNN
 F 3 "~" H 7100 2200 50  0001 C CNN
 	1    7100 2200
@@
 F 0 "R215" V 7100 2950 50  0000 C CNN
 F 1 "10R" V 6984 3000 50  0000 C CNN
-F 2 "Resistor_SMD:R_0805_2012Metric_Pad1.15x1.40mm_HandSolder" V 7030 3000 50  0001 C CNN
+F 2 "AJ:R_0805_2012Metric_Pad1.15x1.40mm_HandSolder" V 7030 3000 50  0001 C CNN
 F 3 "~" H 7100 3000 50  0001 C CNN
 	1    7100 3000
@@
 F 0 "D207" V 6125 3025 50  0000 R CNN
 F 1 "On LED" V 6050 3075 50  0000 R CNN
-F 2 "LED_SMD:LED_0805_2012Metric" H 6050 2800 50  0001 C CNN
+F 2 "AJ:D_0805_2012Metric_Pad1.15x1.40mm_HandSolder" H 6050 2800 50  0001 C CNN
 F 3 "~" H 6050 2800 50  0001 C CNN
 	1    6050 2800
@@
 F 0 "R213" V 6225 2600 50  0000 C CNN
 F 1 "10k" V 6325 2600 50  0000 C CNN
-F 2 "Resistor_SMD:R_0805_2012Metric_Pad1.15x1.40mm_HandSolder" V 6155 2600 50  0001 C CNN
+F 2 "AJ:R_0805_2012Metric_Pad1.15x1.40mm_HandSolder" V 6155 2600 50  0001 C CNN
 F 3 "~" H 6225 2600 50  0001 C CNN
 	1    6225 2600
@@
 F 0 "C207" H 1765 4646 50  0000 L CNN
 F 1 "47n" H 1765 4555 50  0000 L CNN
-F 2 "Capacitor_SMD:C_0805_2012Metric_Pad1.15x1.40mm_HandSolder" H 1688 4450 50  0001 C CNN
+F 2 "AJ:C_0805_2012Metric_Pad1.15x1.40mm_HandSolder" H 1688 4450 50  0001 C CNN
 F 3 "~" H 1650 4600 50  0001 C CNN
 	1    1650 4600
@@
 F 0 "R212" V 1200 4525 50  0000 C CNN
 F 1 "10k" V 1084 4500 50  0000 C CNN
-F 2 "Resistor_SMD:R_0805_2012Metric_Pad1.15x1.40mm_HandSolder" V 1130 4500 50  0001 C CNN
+F 2 "AJ:R_0805_2012Metric_Pad1.15x1.40mm_HandSolder" V 1130 4500 50  0001 C CNN
 F 3 "~" H 1200 4500 50  0001 C CNN
 	1    1200 4500

Commit message: AJ footprints updated
Parts:
- C202, C203, C205, C207: footprint AJ:C_0805_2012Metric_Pad1.15x1.40mm_HandSolder -> AJ:C_0805_AJ
- D207: footprint AJ:D_0805_2012Metric_Pad1.15x1.40mm_HandSolder -> AJ:D_0805_AJ
- R201, R202, R203, R204, R205, R206, R207, R208, R209, R210, R211, R212, R213, R214, R215: footprint AJ:R_0805_2012Metric_Pad1.15x1.40mm_HandSolder -> AJ:R_0805_AJ
Changed lines of the file:
@@
 F 0 "R204" V 1400 3550 50  0000 C CNN
 F 1 "10k" V 1284 3550 50  0000 C CNN
-F 2 "AJ:R_0805_2012Metric_Pad1.15x1.40mm_HandSolder" V 1330 3550 50  0001 C CNN
+F 2 "AJ:R_0805_AJ" V 1330 3550 50  0001 C CNN
 F 3 "~" H 1400 3550 50  0001 C CNN
 	1    1400 3550
@@
 F 0 "R205" V 1400 3950 50  0000 C CNN
 F 1 "1k" V 1500 3950 50  0000 C CNN
-F 2 "AJ:R_0805_2012Metric_Pad1.15x1.40mm_HandSolder" V 1330 3950 50  0001 C CNN
+F 2 "AJ:R_0805_AJ" V 1330 3950 50  0001 C CNN
 F 3 "~" H 1400 3950 50  0001 C CNN
 	1    1400 3950
@@
 F 0 "R207" V 1400 4400 50  0000 C CNN
 F 1 "10k" V 1500 4400 50  0000 C CNN
-F 2 "AJ:R_0805_2012Metric_Pad1.15x1.40mm_HandSolder" V 1330 4400 50  0001 C CNN
+F 2 "AJ:R_0805_AJ" V 1330 4400 50  0001 C CNN
 F 3 "~" H 1400 4400 50  0001 C CNN
 	1    1400 4400
@@
 F 0 "R209" V 1400 4850 50  0000 C CNN
 F 1 "47k" V 1284 4850 50  0000 C CNN
-F 2 "AJ:R_0805_2012Metric_Pad1.15x1.40mm_HandSolder" V 1330 4850 50  0001 C CNN
+F 2 "AJ:R_0805_AJ" V 1330 4850 50  0001 C CNN
 F 3 "~" H 1400 4850 50  0001 C CNN
 	1    1400 4850
@@
 F 0 "R206" V 1800 4150 50  0000 C CNN
 F 1 "100k" V 1684 4200 50  0000 C CNN
-F 2 "AJ:R_0805_2012Metric_Pad1.15x1.40mm_HandSolder" V 1730 4200 50  0001 C CNN
+F 2 "AJ:R_0805_AJ" V 1730 4200 50  0001 C CNN
 F 3 "~" H 1800 4200 50  0001 C CNN
 	1    1800 4200
@@
 F 0 "R210" V 2950 4800 50  0000 C CNN
 F 1 "4k7" V 2834 4850 50  0000 C CNN
-F 2 "AJ:R_0805_2012Metric_Pad1.15x1.40mm_HandSolder" V 2880 4850 50  0001 C CNN
+F 2 "AJ:R_0805_AJ" V 2880 4850 50  0001 C CNN
 F 3 "~" H 2950 4850 50  0001 C CNN
 	1    2950 4850
@@
 F 0 "R211" V 2950 5100 50  0000 C CNN
 F 1 "OPEN" V 2834 5150 50  0000 C CNN
-F 2 "AJ:R_0805_2012Metric_Pad1.15x1.40mm_HandSolder" V 2880 5150 50  0001 C CNN
+F 2 "AJ:R_0805_AJ" V 2880 5150 50  0001 C CNN
 F 3 "~" H 2950 5150 50  0001 C CNN
 	1    2950 5150
@@
 F 0 "C202" H 2665 2096 50  0000 L CNN
 F 1 "10n" H 2665 2005 50  0000 L CNN
-F 2 "AJ:C_0805_2012Metric_Pad1.15x1.40mm_HandSolder" H 2588 1900 50  0001 C CNN
+F 2 "AJ:C_0805_AJ" H 2588 1900 50  0001 C CNN
 F 3 "~" H 2550 2050 50  0001 C CNN
 	1    2550 2050
@@
 F 0 "R203" V 1650 3300 50  0000 C CNN
 F 1 "100k" V 1534 3350 50  0000 C CNN
-F 2 "AJ:R_0805_2012Metric_Pad1.15x1.40mm_HandSolder" V 1580 3350 50  0001 C CNN
+F 2 "AJ:R_0805_AJ" V 1580 3350 50  0001 C CNN
 F 3 "~" H 1650 3350 50  0001 C CNN
 	1    1650 3350
@@
 F 0 "R208" V 1850 5000 50  0000 C CNN
 F 1 "100k" V 1750 5150 50  0000 C CNN
-F 2 "AJ:R_0805_2012Metric_Pad1.15x1.40mm_HandSolder" V 1780 5050 50  0001 C CNN
+F 2 "AJ:R_0805_AJ" V 1780 5050 50  0001 C CNN
 F 3 "~" H 1850 5050 50  0001 C CNN
 	1    1850 5050
@@
 F 0 "R202" V 2150 1450 50  0000 C CNN
 F 1 "220k" V 2034 1450 50  0000 C CNN
-F 2 "AJ:R_0805_2012Metric_Pad1.15x1.40mm_HandSolder" V 2080 1450 50  0001 C CNN
+F 2 "AJ:R_0805_AJ" V 2080 1450 50  0001 C CNN
 F 3 "~" H 2150 1450 50  0001 C CNN
 	1    2150 1450
@@
 F 0 "R201" V 4150 1100 50  0000 C CNN
 F 1 "3k3" V 4034 1150 50  0000 C CNN
-F 2 "AJ:R_0805_2012Metric_Pad1.15x1.40mm_HandSolder" V 4080 1150 50  0001 C CNN
+F 2 "AJ:R_0805_AJ" V 4080 1150 50  0001 C CNN
 F 3 "~" H 4150 1150 50  0001 C CNN
 	1    4150 1150
@@
 F 0 "C203" H 7465 2446 50  0000 L CNN
 F 1 "1u" H 7465 2355 50  0000 L CNN
-F 2 "AJ:C_0805_2012Metric_Pad1.15x1.40mm_HandSolder" H 7388 2250 50  0001 C CNN
+F 2 "AJ:C_0805_AJ" H 7388 2250 50  0001 C CNN
 F 3 "~" H 7350 2400 50  0001 C CNN
 	1    7350 2400
@@
 F 0 "C205" H 8065 2446 50  0000 L CNN
 F 1 "1u" H 8065 2355 50  0000 L CNN
-F 2 "AJ:C_0805_2012Metric_Pad1.15x1.40mm_HandSolder" H 7988 2250 50  0001 C CNN
+F 2 "AJ:C_0805_AJ" H 7988 2250 50  0001 C CNN
 F 3 "~" H 7950 2400 50  0001 C CNN
 	1    7950 2400
@@
 F 0 "R214" V 7100 2150 50  0000 C CNN
 F 1 "10R" V 6984 2200 50  0000 C CNN
-F 2 "AJ:R_0805_2012Metric_Pad1.15x1.40mm_HandSolder" V 7030 2200 50  0001 C CNN
+F 2 "AJ:R_0805_AJ" V 7030 2200 50  0001 C CNN
 F 3 "~" H 7100 2200 50  0001 C CNN
 	1    7100 2200
@@
 F 0 "R215" V 7100 2950 50  0000 C CNN
 F 1 "10R" V 6984 3000 50  0000 C CNN
-F 2 "AJ:R_0805_2012Metric_Pad1.15x1.40mm_HandSolder" V 7030 3000 50  0001 C CNN
+F 2 "AJ:R_0805_AJ" V 7030 3000 50  0001 C CNN
 F 3 "~" H 7100 3000 50  0001 C CNN
 	1    7100 3000
@@
 F 0 "D207" V 6125 3025 50  0000 R CNN
 F 1 "On LED" V 6050 3075 50  0000 R CNN
-F 2 "AJ:D_0805_2012Metric_Pad1.15x1.40mm_HandSolder" H 6050 2800 50  0001 C CNN
+F 2 "AJ:D_0805_AJ" H 6050 2800 50  0001 C CNN
 F 3 "~" H 6050 2800 50  0001 C CNN
 	1    6050 2800
@@
 F 0 "R213" V 6225 2600 50  0000 C CNN
 F 1 "10k" V 6325 2600 50  0000 C CNN
-F 2 "AJ:R_0805_2012Metric_Pad1.15x1.40mm_HandSolder" V 6155 2600 50  0001 C CNN
+F 2 "AJ:R_0805_AJ" V 6155 2600 50  0001 C CNN
 F 3 "~" H 6225 2600 50  0001 C CNN
 	1    6225 2600
@@
 F 0 "C207" H 1765 4646 50  0000 L CNN
 F 1 "47n" H 1765 4555 50  0000 L CNN
-F 2 "AJ:C_0805_2012Metric_Pad1.15x1.40mm_HandSolder" H 1688 4450 50  0001 C CNN
+F 2 "AJ:C_0805_AJ" H 1688 4450 50  0001 C CNN
 F 3 "~" H 1650 4600 50  0001 C CNN
 	1    1650 4600
@@
 F 0 "R212" V 1200 4525 50  0000 C CNN
 F 1 "10k" V 1084 4500 50  0000 C CNN
-F 2 "AJ:R_0805_2012Metric_Pad1.15x1.40mm_HandSolder" V 1130 4500 50  0001 C CNN
+F 2 "AJ:R_0805_AJ" V 1130 4500 50  0001 C CNN
 F 3 "~" H 1200 4500 50  0001 C CNN
 	1    1200 4500

Commit message: hold/rst
Connections:
- net clk: now reaches J205.1 (Pin_1), U202.14 (CLK)
Changed lines of the file:
@@
 Wire Wire Line
 	8150 3000 8325 3000
+Text Label 2875 3600 0    50   ~ 0
+clk
 $EndSCHEMATC
